File: KiCAD/LiF_FC-PCB_rev1/01_Buttons.kicad_sch (KiCad schematic)
At the start: 0 parts

Commit message: fixed my schematics syncing (I think), and added accelorometer schematic. Pushing since I need to switch main.
Parts:
- added D? (x8): LED, LED_SMD:LED_0805_2012Metric_Pad1.15x1.40mm_HandSolder, symbol Device:LED
- added R? (x7): 10k, Resistor_SMD:R_0805_2012Metric, symbol Device:R
- added R?: EXB-2HV471JV, RES_EXB2HV, symbol EXB-2HV471JV:EXB-2HV471JV
- added S? (x7): TL3301PF160QG, TL3301PF160QG:SW_TL3301PF160QG, symbol TL3301PF160QG:TL3301PF160QG
- added U?: 74HCT595, 74HC595PW_118:SOP65P640X110-16N, symbol 74xx:74HCT595
Connections:
- new net: D?.2 (A), R?.13
- new net: R?.2, S?.1 (x7)
- new net: R?.2, U?.1 (QB)
- new net: R?.1, U?.15 (QA)
- new net: R?.3, U?.2 (QC)
- new net: R?.4, U?.3 (QD)
- new net: R?.5, U?.4 (QE)
- new net: R?.6, U?.5 (QF)
- new net: R?.7, U?.6 (QG)
- new net: R?.8, U?.7 (QH)
- new net: D?.2 (A), R?.9
- new net: D?.2 (A), R?.16
- new net: D?.2 (A), R?.14
- new net: D?.2 (A), R?.12
- new net: D?.2 (A), R?.15
- new net: D?.2 (A), R?.10
- new net: D?.2 (A), R?.11
- new net +3.3V: R?.1, R?.1, R?.1, R?.1, R?.1, R?.1, R?.1, U?.10 (~{SRCLR}), U?.16 (VCC)
- new net ESP_CLK: U?.11 (SRCLK)
- new net ESP_DATA: U?.14 (SER)
- new net ESP_LATCH: U?.12 (RCLK)
- new net GND: D?.1 (K), D?.1 (K), D?.1 (K), D?.1 (K), D?.1 (K), D?.1 (K), D?.1 (K), D?.1 (K), S?.3, S?.3, S?.3, S?.3, S?.3, S?.3, S?.3, U?.13 (~{OE}), U?.8 (GND)
- no-connect marks 0 -> 1
Other:
- note added: "ENCODER MODULE - SEND COMMAND"
- note added: "Floor 1"
- note added: "Floor 2"
- note added: "Floor 3"
- note added: "Floor 4"
- note added: "Floor 5"
- note added: "Floor 6"
- note added: "Floor 7/Spare"
- note added: "From any ESP GPIO"
- note added: "Sheet 04 - User Interface Button and LED Array"
- company: (none) -> Conestoga College
- title: (none) -> LiF - PD, UI, and Audio

Commit message: updated schematics and pushing so MR can pull and begin merge.
Parts:
- gave numbers to parts that had none: 23
Connections:
- net FLOOR5: now reaches R04_05.2, S5.1
- net FLOOR4: now reaches R04_04.2, S4.1
- net SPARE/CC: now reaches R04_07.2, S7.1
- net FLOOR6: now reaches R04_06.2, S6.1
- net FLOOR2: now reaches R04_02.2, S2.1
- net FLOOR1: now reaches R04_01.2, S1.1
- net FLOOR3: now reaches R04_03.2, S3.1
- net ESP_CLK renamed ESP_PBLED_CLK
- net ESP_DATA renamed ESP_PBLED_DATA
- net ESP_LATCH renamed ESP_PBLED_LATCH
Other:
- note added: "Buttons can be whatever, but I used tall ones found here: https://www.digikey.ca/en/products/detail/e-switch/tl3301pf160qg/1756542 Also, for resistor it may be worth using an array. I designed this before I knew what R-arr's looked like. Here's a link to one I found that's 10k and has 8 resistors: https://www.digikey.ca/en/products/detail/panasonic-industry/EXB-2HV103JV/285331 Additionally, inste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"
- note added: "You'll probably have to add a footprint for this one... (74HCT595) There are SOIC-16 and TSSOP-16 options available on DigiKey. Links below: TSSOP-16: https://www.digikey.ca/en/products/detail/nexperia-usa-inc/74HCT595PW-118/763165 SOIC-16: https://www.digikey.ca/en/products/detail/nexperia-usa-inc/74HCT595D-118/763163 So use whatever footprint you prefer"
