File: KiCAD/LiF_FC-PCB_rev1/01_PD_Source.kicad_sch (KiCad schematic)
At the start: 0 parts

Commit message: fixed my schematics syncing (I think), and added accelorometer schematic. Pushing since I need to switch main.
Other:
- company: (none) -> Conestoga College
- title: (none) -> LiF - PD, UI, and Audio
Changed lines of the file:
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@@
 	(generator_version "9.0")
 	(paper "A4")
+	(title_block
+		(title "LiF - PD, UI, and Audio")
+		(date "2026-07-02")
+		(rev "0")
+		(company "Conestoga College")
+		(comment 1 "Designed by NK")
+	)
 )

Commit message: updated schematics and pushing so MR can pull and begin merge.
Other:
- note added: "yo mama"
Changed lines of the file:
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@@
 		(comment 1 "Designed by NK")
 	)
+	(text "yo mama"
+		(exclude_from_sim no)
+		(at 151.13 93.726 0)
+		(effects
+			(font
+				(size 1.27 1.27)
+			)
+			(justify left)
+		)
+	)
 )
