File: KiCAD/LiF_FC-PCB_rev1/02_PD_Sink.kicad_sch (KiCad schematic)
At the start: 0 parts

Commit message: fixed my schematics syncing (I think), and added accelorometer schematic. Pushing since I need to switch main.
Parts:
- added C?: 1uF, Capacitor_SMD:C_0805_2012Metric, symbol Device:C
- added R6: 1k, Resistor_SMD:R_0805_2012Metric, symbol Device:R
- added R7: 10k, Resistor_SMD:R_0805_2012Metric, symbol Device:R
- added R8: 56k, Resistor_SMD:R_0805_2012Metric, symbol Device:R
- added U4: CH224K, Package_SO:SSOP-10-1EP_3.9x4.9mm_P1mm_EP2.1x3.3mm, symbol Interface_USB:CH224K
Connections:
- new net: C?.2, R6.2, U4.1 (VDD)
- new net: R7.2, U4.8 (VBUS)
- new net: R8.1, U4.9 (CFG1)
- new net GND: C?.1, R8.2, U4.11 (GND)
- new net PD_VBus: R6.1, R7.1
- new net USBC_IN_CC1: U4.7 (CC1)
- new net USBC_IN_CC2: U4.6 (CC2)
- no-connect marks 0 -> 5
Other:
- note added: "15V rail for regulation"
- note added: "Configured VBus to be 15V. 6.8k = 9V 24k = 12V 56k = 15V NC = 20V"
- note added: "DP/DM are D+/D- Used by CANbus so NC here"
- note added: "Sheet 02 - Power Delivery PD Sink"
- company: (none) -> Conestoga College
- title: (none) -> LiF - PD, UI, and Audio

Commit message: updated schematics and pushing so MR can pull and begin merge.
Parts:
- gave numbers to parts that had none: 1
- renumbered R6 to R02_01, R7 to R02_02, R8 to R02_03, U4 to U1
Other:
- note added: "Configured VBus to be 15V. See datasheet in my logbook (2026-07-03) 6.8k = 9V 24k = 12V 56k = 15V NC = 20V"
- note removed: "Configured VBus to be 15V. 6.8k = 9V 24k = 12V 56k = 15V NC = 20V"
Changed lines of the file:
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@@
 		)
 	)
-	(text "Configured VBus to be 15V.\n\n6.8k = 9V\n24k = 12V\n56k = 15V\nNC = 20V"
+	(text "Configured VBus to be 15V. \nSee datasheet in my logbook (2026-07-03)\n\n6.8k = 9V\n24k = 12V\n56k = 15V\nNC = 20V"
 		(exclude_from_sim no)
 		(at 142.748 88.646 0)
@@
 	(text "DP/DM are D+/D-\n\nUsed by CANbus so NC here"
 		(exclude_from_sim no)
-		(at 95.25 88.138 0)
+		(at 94.742 88.138 0)
 		(effects
 			(font
@@
 		)
 	)
-	(global_label "PD_VBus"
+	(hierarchical_label "USBC_IN_CC2"
+		(shape input)
+		(at 66.04 80.01 180)
+		(effects
+			(font
+				(size 1.27 1.27)
+			)
+			(justify right)
+		)
+	)
+	(hierarchical_label "PD_VBus"
 		(shape input)
 		(at 140.97 55.88 0)
-		(fields_autoplaced yes)
 		(effects
 			(font
@@
 			(justify left)
 		)
-		(property "Intersheetrefs" "${INTERSHEET_REFS}"
-			(at 151.9985 55.88 0)
-			(effects
-				(font
-					(size 1.27 1.27)
-				)
-				(justify left)
-				(hide yes)
-			)
-		)
-	)
-	(global_label "USBC_IN_CC1"
+	)
+	(hierarchical_label "USBC_IN_CC1"
 		(shape input)
 		(at 66.04 77.47 180)
-		(fields_autoplaced yes)
 		(effects
 			(font
@@
 			(justify right)
 		)
-		(property "Intersheetrefs" "${INTERSHEET_REFS}"
-			(at 50.3548 77.47 0)
-			(effects
-				(font
-					(size 1.27 1.27)
-				)
-				(justify right)
-				(hide yes)
-			)
-		)
-	)
-	(global_label "USBC_IN_VBus"
+	)
+	(hierarchical_label "USBC_IN_VBus"
 		(shape input)
 		(at 64.77 55.88 180)
-		(fields_autoplaced yes)
 		(effects
 			(font
@@
 			)
 			(justify right)
-		)
-		(property "Intersheetrefs" "${INTERSHEET_REFS}"
-			(at 48.2986 55.88 0)
-			(effects
-				(font
-					(size 1.27 1.27)
-				)
-				(justify right)
-				(hide yes)
-			)
-		)
-	)
-	(global_label "USBC_IN_CC2"
-		(shape input)
-		(at 66.04 80.01 180)
-		(fields_autoplaced yes)
-		(effects
-			(font
-				(size 1.27 1.27)
-			)
-			(justify right)
-		)
-		(property "Intersheetrefs" "${INTERSHEET_REFS}"
-			(at 50.3548 80.01 0)
-			(effects
-				(font
-					(size 1.27 1.27)
-				)
-				(justify right)
-				(hide yes)
-			)
 		)
 	)
@@
 		(on_board yes)
 		(dnp no)
-		(property "Reference" "R6"
+		(property "Reference" "R02_01"
 			(at 83.82 59.944 90)
 			(effects
@@
 			(project "LiF_CustomPCB"
 				(path "/e8d53809-63ab-4a8d-88b7-d7504d15b103/8daafc21-1287-4370-9327-711e48673ef9"
-					(reference "R6")
+					(reference "R02_01")
 					(unit 1)
 				)
@@
 		(dnp no)
 		(fields_autoplaced yes)
-		(property "Reference" "C?"
+		(property "Reference" "C02_01"
 			(at 97.79 64.7699 0)
 			(effects
@@
 			(project "LiF_CustomPCB"
 				(path "/e8d53809-63ab-4a8d-88b7-d7504d15b103/8daafc21-1287-4370-9327-711e48673ef9"
-					(reference "C?")
+					(reference "C02_01")
 					(unit 1)
 				)
@@
 		(on_board yes)
 		(dnp no)
-		(property "Reference" "R7"
-			(at 114.3 65.532 0)
+		(property "Reference" "R02_02"
+			(at 115.316 65.532 0)
 			(effects
 				(font
@@
 			(project "LiF_CustomPCB"
 				(path "/e8d53809-63ab-4a8d-88b7-d7504d15b103/8daafc21-1287-4370-9327-711e48673ef9"
-					(reference "R7")
+					(reference "R02_02")
 					(unit 1)
 				)
@@
 		(on_board yes)
 		(dnp no)
-		(property "Reference" "R8"
-			(at 136.398 89.154 0)
+		(property "Reference" "R02_03"
+			(at 134.874 89.408 0)
 			(effects
 				(font
@@
 			(project "LiF_CustomPCB"
 				(path "/e8d53809-63ab-4a8d-88b7-d7504d15b103/8daafc21-1287-4370-9327-711e48673ef9"
-					(reference "R8")
+					(reference "R02_03")
 					(unit 1)
 				)
@@
 		(dnp no)
 		(fields_autoplaced yes)
-		(property "Reference" "U4"
+		(property "Reference" "U1"
 			(at 110.0933 92.71 0)
 			(effects
@@
 			(project "LiF_CustomPCB"
 				(path "/e8d53809-63ab-4a8d-88b7-d7504d15b103/8daafc21-1287-4370-9327-711e48673ef9"
-					(reference "U4")
+					(reference "U1")
 					(unit 1)
 				)
