File: KiCAD/LiF_FC-PCB_rev1/03_SevenSegment.kicad_sch (KiCad schematic)
At the start: 0 parts

Commit message: fixed my schematics syncing (I think), and added accelorometer schematic. Pushing since I need to switch main.
Parts:
- added R1, R2: EXB-2HV471JV, RES_EXB2HV, symbol EXB-2HV471JV:EXB-2HV471JV
- added U1, U2: 74HCT595, 74HC595PW_118:SOP65P640X110-16N, symbol 74xx:74HCT595
- added U3: DC56-11EWA, Display_7Segment:DA56-11SURKWA, symbol Display_Character:DC56-11EWA
Connections:
- new net: R2.1, U2.15 (QA)
- new net: R2.10, U3.7 (DIG2_G)
- new net: R2.11, U3.12 (DIG2_F)
- new net: R2.12, U3.5 (DIG2_E)
- new net: R2.13, U3.6 (DIG2_D)
- new net: R2.14, U3.8 (DIG2_C)
- new net: R2.15, U3.10 (DIG2_B)
- new net: R2.16, U3.11 (DIG2_A)
- new net: R2.2, U2.1 (QB)
- new net: R2.3, U2.2 (QC)
- new net: R2.4, U2.3 (QD)
- new net: R2.5, U2.4 (QE)
- new net: R2.6, U2.5 (QF)
- new net: R2.7, U2.6 (QG)
- new net: R2.8, U2.7 (QH)
- new net: R2.9, U3.9 (DP2)
- new net: R1.12, U3.1 (DIG1_E)
- new net: R1.15, U3.15 (DIG1_B)
- new net: R1.16, U3.16 (DIG1_A)
- new net: R1.10, U3.17 (DIG1_G)
- new net: R1.11, U3.18 (DIG1_F)
- new net: R1.13, U3.2 (DIG1_D)
- new net: R1.14, U3.3 (DIG1_C)
- new net: R1.9, U3.4 (DP1)
- new net: R1.1, U1.15 (QA)
- new net: R1.2, U1.1 (QB)
- new net: R1.3, U1.2 (QC)
- new net: R1.4, U1.3 (QD)
- new net: R1.5, U1.4 (QE)
- new net: R1.6, U1.5 (QF)
- new net: R1.7, U1.6 (QG)
- new net: R1.8, U1.7 (QH)
- new net +3.3V: U1.10 (~{SRCLR}), U1.16 (VCC), U2.10 (~{SRCLR}), U2.16 (VCC)
- new net Data Chain: U1.9 (QH'), U2.14 (SER), U2.9 (QH')
- new net ESP_CLK: U1.11 (SRCLK), U2.11 (SRCLK)
- new net ESP_DATA: U1.14 (SER)
- new net ESP_LATCH: U1.12 (RCLK), U2.12 (RCLK)
- new net GND: U1.13 (~{OE}), U1.8 (GND), U2.13 (~{OE}), U2.8 (GND), U3.13 (DIG2_CC), U3.14 (DIG1_CC)
Other:
- note added: "7 SEGMENT MODULE"
- note added: "From any ESP GPIO"
- note added: "Sheet 05 - User Interface Shift Registers and Seven Segment Displays"
- company: (none) -> Conestoga College
- title: (none) -> LiF - PD, UI, and Audio

Commit message: updated schematics and pushing so MR can pull and begin merge.
Parts:
- renumbered R1 to R05_Array01, R2 to R05_Array02, U1 to U2, U2 to U3, U3 to U4
Connections:
- net Data Chain: no longer U3.9 (QH')
- net ESP_CLK renamed ESP_SEVSEG_CLK
- net ESP_DATA renamed ESP_SEVSEG_DATA
- net ESP_LATCH renamed ESP_SEVSEG_LATCH
- no-connect marks 0 -> 1
Other:
- note added: "For resistor array footprints, see the DigiKey part here: https://www.digikey.ca/en/products/detail/panasonic-industry/EXB-2HV471JV/285315?s=N4IgTCBcDaIKIA0BCBaMAJAagFgOwEYApTEAXQF8g"
- note added: "You'll probably have to add a footprint for this one... (74HCT595) There are SOIC-16 and TSSOP-16 options available on DigiKey. Links below: TSSOP-16: https://www.digikey.ca/en/products/detail/nexperia-usa-inc/74HCT595PW-118/763165 SOIC-16: https://www.digikey.ca/en/products/detail/nexperia-usa-inc/74HCT595D-118/763163 So use whatever footprint you prefer"
Changed lines of the file:
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@@
 	)
 	(rectangle
-		(start 28.575 33.655)
-		(end 242.57 159.385)
+		(start 20.32 33.655)
+		(end 258.445 159.385)
 		(stroke
 			(width 0)
@@
 		)
 	)
+	(text "You'll probably have to add a footprint for this one... (74HCT595)\n\nThere are SOIC-16 and TSSOP-16 options available on DigiKey. Links below:\n\nTSSOP-16:\nhttps://www.digikey.ca/en/products/detail/nexperia-usa-inc/74HCT595PW-118/763165\n\n\nSOIC-16:\nhttps://www.digikey.ca/en/products/detail/nexperia-usa-inc/74HCT595D-118/763163\n\n\nSo use whatever footprint you prefer"
+		(exclude_from_sim no)
+		(at 28.194 175.514 0)
+		(effects
+			(font
+				(size 1.27 1.27)
+			)
+			(justify left)
+		)
+	)
 	(text "From any\nESP GPIO\n"
 		(exclude_from_sim no)
@@
 		)
 	)
+	(text "For resistor array footprints, see the DigiKey part here:\n\n\nhttps://www.digikey.ca/en/products/detail/panasonic-industry/EXB-2HV471JV/285315?s=N4IgTCBcDaIKIA0BCBaMAJAagFgOwEYApTEAXQF8g"
+		(exclude_from_sim no)
+		(at 112.014 40.132 0)
+		(effects
+			(font
+				(size 1.27 1.27)
+			)
+			(justify left)
+		)
+	)
 	(text "Sheet 05 - User Interface\n\nShift Registers and Seven Segment Displays"
 		(exclude_from_sim no)
@@
 		(color 0 0 0 0)
 	)
+	(no_connect
+		(at 80.01 142.24)
+	)
 	(wire
 		(pts
@@
 	(wire
 		(pts
-			(xy 80.01 142.24) (xy 80.01 157.48)
-		)
-		(stroke
-			(width 0)
-			(type default)
-		)
-	)
-	(wire
-		(pts
 			(xy 90.17 72.39) (xy 95.25 72.39)
 		)
@@
 		(pts
 			(xy 87.63 71.12) (xy 87.63 77.47)
-		)
-		(stroke
-			(width 0)
-			(type default)
-		)
-	)
-	(wire
-		(pts
-			(xy 78.74 157.48) (xy 80.01 157.48)
 		)
 		(stroke
@@
 		)
 	)
-	(label "Data Chain"
-		(at 78.74 157.48 180)
+	(hierarchical_label "ESP_SEVSEG_CLK"
+		(shape input)
+		(at 43.18 60.96 180)
 		(effects
 			(font
 				(size 1.27 1.27)
 			)
-			(justify right bottom)
-		)
-	)
-	(global_label "ESP_CLK"
+			(justify right)
+		)
+	)
+	(hierarchical_label "ESP_SEVSEG_LATCH"
 		(shape input)
-		(at 46.99 124.46 180)
-		(fields_autoplaced yes)
+		(at 43.18 68.58 180)
 		(effects
 			(font
@@
 			(justify right)
 		)
-		(property "Intersheetrefs" "${INTERSHEET_REFS}"
-			(at 35.8406 124.46 0)
-			(effects
-				(font
-					(size 1.27 1.27)
-				)
-				(justify right)
-				(hide yes)
-			)
-		)
-	)
-	(global_label "ESP_LATCH"
+	)
+	(hierarchical_label "ESP_SEVSEG_DATA"
 		(shape input)
-		(at 43.18 68.58 180)
-		(fields_autoplaced yes)
+		(at 43.18 55.88 180)
 		(effects
 			(font
@@
 			(justify right)
 		)
-		(property "Intersheetrefs" "${INTERSHEET_REFS}"
-			(at 29.9139 68.58 0)
-			(effects
-				(font
-					(size 1.27 1.27)
-				)
-				(justify right)
-				(hide yes)
-			)
-		)
-	)
-	(global_label "ESP_DATA"
+	)
+	(hierarchical_label "ESP_SEVSEG_LATCH"
 		(shape input)
-		(at 43.18 55.88 180)
-		(fields_autoplaced yes)
+		(at 46.99 132.08 180)
 		(effects
 			(font
@@
 			(justify right)
 		)
-		(property "Intersheetrefs" "${INTERSHEET_REFS}"
-			(at 31.1839 55.88 0)
-			(effects
-				(font
-					(size 1.27 1.27)
-				)
-				(justify right)
-				(hide yes)
-			)
-		)
-	)
-	(global_label "ESP_CLK"
+	)
+	(hierarchical_label "ESP_SEVSEG_CLK"
 		(shape input)
-		(at 43.18 60.96 180)
-		(fields_autoplaced yes)
+		(at 46.99 124.46 180)
 		(effects
 			(font
@@
 			)
 			(justify right)
-		)
-		(property "Intersheetrefs" "${INTERSHEET_REFS}"
-			(at 32.0306 60.96 0)
-			(effects
-				(font
-					(size 1.27 1.27)
-				)
-				(justify right)
-				(hide yes)
-			)
-		)
-	)
-	(global_label "ESP_LATCH"
-		(shape input)
-		(at 46.99 132.08 180)
-		(fields_autoplaced yes)
-		(effects
-			(font
-				(size 1.27 1.27)
-			)
-			(justify right)
-		)
-		(property "Intersheetrefs" "${INTERSHEET_REFS}"
-			(at 33.7239 132.08 0)
-			(effects
-				(font
-					(size 1.27 1.27)
-				)
-				(justify right)
-				(hide yes)
-			)
 		)
 	)
@@
 		(dnp no)
 		(fields_autoplaced yes)
-		(property "Reference" "R2"
+		(property "Reference" "R05_Array02"
 			(at 105.41 104.14 0)
 			(effects
@@
 			(project "LiF_CustomPCB"
 				(path "/e8d53809-63ab-4a8d-88b7-d7504d15b103/4d480ead-5d90-4d49-ad2d-4ec0e23f6f32"
-					(reference "R2")
+					(reference "R05_Array02")
 					(unit 1)
 				)
@@
 		(dnp no)
 		(fields_autoplaced yes)
-		(property "Reference" "U3"
+		(property "Reference" "U4"
 			(at 173.99 67.31 0)
 			(effects
@@
 			(project "LiF_CustomPCB"
 				(path "/e8d53809-63ab-4a8d-88b7-d7504d15b103/4d480ead-5d90-4d49-ad2d-4ec0e23f6f32"
-					(reference "U3")
+					(reference "U4")
 					(unit 1)
 				)
@@
 		(dnp no)
 		(fields_autoplaced yes)
-		(property "Reference" "R1"
+		(property "Reference" "R05_Array01"
 			(at 101.6 40.64 0)
 			(effects
@@
 			(project "LiF_CustomPCB"
 				(path "/e8d53809-63ab-4a8d-88b7-d7504d15b103/4d480ead-5d90-4d49-ad2d-4ec0e23f6f32"
-					(reference "R1")
+					(reference "R05_Array01")
 					(unit 1)
 				)
@@
 		(dnp no)
 		(fields_autoplaced yes)
-		(property "Reference" "U2"
+		(property "Reference" "U3"
 			(at 69.4533 111.76 0)
 			(effects
@@
 			(project "LiF_CustomPCB"
 				(path "/e8d53809-63ab-4a8d-88b7-d7504d15b103/4d480ead-5d90-4d49-ad2d-4ec0e23f6f32"
-					(reference "U2")
+					(reference "U3")
 					(unit 1)
 				)
@@
 		(dnp no)
 		(fields_autoplaced yes)
-		(property "Reference" "U1"
+		(property "Reference" "U2"
 			(at 65.6433 48.26 0)
 			(effects
@@
 			(project "LiF_CustomPCB"
 				(path "/e8d53809-63ab-4a8d-88b7-d7504d15b103/4d480ead-5d90-4d49-ad2d-4ec0e23f6f32"
-					(reference "U1")
+					(reference "U2")
 					(unit 1)
 				)
