File: KiCAD/LiF_FC-PCB_rev1/Encoder.kicad_sch (KiCad schematic)
At the start: 0 parts

Commit message: fixed my schematics syncing (I think), and added accelorometer schematic. Pushing since I need to switch main.
Parts:
- added MT?: PEC11R-4215F-S0024, PEC11R_4215F_S0024:XDCR_PEC11R-4215F-S0024, symbol PEC11R-4215F-S0024:PEC11R-4215F-S0024
- added R3, R4, R5: 10k, Resistor_SMD:R_0805_2012Metric, symbol Device:R
Connections:
- new net +3.3V: R3.1, R4.1, R5.1
- new net ENC_A: MT?.A, R4.2
- new net ENC_B: MT?.B, R5.2
- new net ENC_SW: MT?.2, R3.2
- new net GND: MT?.1, MT?.COM, MT?.S1 (SHIELD), MT?.S2 (SHIELD__1)
Other:
- note added: "ENCODER MODULE - FLOOR SELECTOR"
- note added: "Function (car controller) Encoder will be rotated and the value will be updated on the 7-seg display. This will be the floor selector Once you picked a floor (say 7), you can click the PB to either send the command directly Or this will function as a queue loader (multi-floor select like a real elevator) with the encoder switch being the send command The LED flashes once when floor queued but glo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"
- note added: "Pull up R's for input"
- note added: "Rotary Encoder"
- note added: "Sheet 03 - User Interface Encoder Module"
- note added: "Shield to GND"
- note added: "To any ESP GPIO"
- company: (none) -> Conestoga College
- title: (none) -> LiF - PD, UI, and Audio

Commit message: updated schematics and pushing so MR can pull and begin merge.
Parts:
- gave numbers to parts that had none: 1
- renumbered R3 to R03_01, R4 to R03_02, R5 to R03_03
Connections:
- net ENC_A renamed Selector_ENCA
- net ENC_B renamed Selector_ENCB
- net ENC_SW renamed Selector_ENC_SW
Other:
- note added: "Function (car controller) Encoder will be rotated and the value will be updated on the 7-seg display. This will behave as a floor selector Delete if not wanted :("
- note removed: "Function (car controller) Encoder will be rotated and the value will be updated on the 7-seg display. This will be the floor selector Once you picked a floor (say 7), you can click the PB to either send the command directly Or this will function as a queue loader (multi-floor select like a real elevator) with the encoder switch being the send command The LED flashes once when floor queued but glo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"
Changed lines of the file:
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@@
 		)
 	)
-	(text "Function (car controller)\nEncoder will be rotated and the value will be updated on the 7-seg display.\nThis will be the floor selector\n\nOnce you picked a floor (say 7), you can click the PB to either send the command directly\nOr this will function as a queue loader (multi-floor select like a real elevator) with the encoder switch being the send command\n\nThe LED flashes once when floor queued but glows when executing commands (like sending CAN out)"
-		(exclude_from_sim no)
-		(at 42.164 112.522 0)
+	(text "Function (car controller)\nEncoder will be rotated and the value will be updated on the 7-seg display.\nThis will behave as a floor selector\n\nDelete if not wanted :("
+		(exclude_from_sim no)
+		(at 41.148 106.172 0)
 		(effects
 			(font
@@
 	(text "To any\nESP GPIO"
 		(exclude_from_sim no)
-		(at 138.684 80.518 0)
+		(at 130.81 90.932 0)
 		(effects
 			(font
@@
 		)
 	)
-	(global_label "ENC_SW"
+	(hierarchical_label "Selector_ENCA"
+		(shape input)
+		(at 123.19 82.55 0)
+		(effects
+			(font
+				(size 1.27 1.27)
+			)
+			(justify left)
+		)
+	)
+	(hierarchical_label "Selector_ENC_SW"
 		(shape input)
 		(at 121.92 77.47 0)
-		(fields_autoplaced yes)
 		(effects
 			(font
@@
 			(justify left)
 		)
-		(property "Intersheetrefs" "${INTERSHEET_REFS}"
-			(at 132.2832 77.47 0)
-			(effects
-				(font
-					(size 1.27 1.27)
-				)
-				(justify left)
-				(hide yes)
-			)
-		)
-	)
-	(global_label "ENC_B"
+	)
+	(hierarchical_label "Selector_ENCB"
 		(shape input)
 		(at 123.19 85.09 0)
-		(fields_autoplaced yes)
 		(effects
 			(font
@@
 			)
 			(justify left)
-		)
-		(property "Intersheetrefs" "${INTERSHEET_REFS}"
-			(at 132.1623 85.09 0)
-			(effects
-				(font
-					(size 1.27 1.27)
-				)
-				(justify left)
-				(hide yes)
-			)
-		)
-	)
-	(global_label "ENC_A"
-		(shape input)
-		(at 123.19 82.55 0)
-		(fields_autoplaced yes)
-		(effects
-			(font
-				(size 1.27 1.27)
-			)
-			(justify left)
-		)
-		(property "Intersheetrefs" "${INTERSHEET_REFS}"
-			(at 131.9809 82.55 0)
-			(effects
-				(font
-					(size 1.27 1.27)
-				)
-				(justify left)
-				(hide yes)
-			)
 		)
 	)
@@
 		(on_board yes)
 		(dnp no)
-		(fields_autoplaced yes)
-		(property "Reference" "R4"
-			(at 110.49 63.4999 0)
+		(property "Reference" "R03_02"
+			(at 108.712 60.452 0)
 			(effects
 				(font
@@
 			(project "LiF_CustomPCB"
 				(path "/e8d53809-63ab-4a8d-88b7-d7504d15b103/e00a619c-d9be-4b49-85f4-4e5c1aa00420"
-					(reference "R4")
+					(reference "R03_02")
 					(unit 1)
 				)
@@
 		(on_board yes)
 		(dnp no)
-		(fields_autoplaced yes)
-		(property "Reference" "R3"
-			(at 100.33 63.4999 0)
+		(property "Reference" "R03_01"
+			(at 98.298 60.706 0)
 			(effects
 				(font
@@
 		)
 		(property "Value" "10k"
-			(at 100.33 66.0399 0)
+			(at 99.568 66.294 0)
 			(effects
 				(font
@@
 			(project "LiF_CustomPCB"
 				(path "/e8d53809-63ab-4a8d-88b7-d7504d15b103/e00a619c-d9be-4b49-85f4-4e5c1aa00420"
-					(reference "R3")
+					(reference "R03_01")
 					(unit 1)
 				)
@@
 		(on_board yes)
 		(dnp no)
-		(fields_autoplaced yes)
-		(property "Reference" "R5"
-			(at 120.65 63.4999 0)
+		(property "Reference" "R03_03"
+			(at 118.872 60.452 0)
 			(effects
 				(font
@@
 			(project "LiF_CustomPCB"
 				(path "/e8d53809-63ab-4a8d-88b7-d7504d15b103/e00a619c-d9be-4b49-85f4-4e5c1aa00420"
-					(reference "R5")
+					(reference "R03_03")
 					(unit 1)
 				)
@@
 		(dnp no)
 		(fields_autoplaced yes)
-		(property "Reference" "MT?"
+		(property "Reference" "MT1"
 			(at 82.55 67.31 0)
 			(effects
@@
 			(project "LiF_CustomPCB"
 				(path "/e8d53809-63ab-4a8d-88b7-d7504d15b103/e00a619c-d9be-4b49-85f4-4e5c1aa00420"
-					(reference "MT?")
+					(reference "MT1")
 					(unit 1)
 				)
