File: KiCAD/LiF_FC-PCB_rev1/LiF_CAN.kicad_sch (KiCad schematic)
At the start: 32 parts, among them J17 Bypass DOWN fuse, J18 CAN Down_{EN}, J19 CAN Upstream, J20 CAN 5V0_{EN}, J21 Bypass OR-ing, J22 Bypass DOWN fuse, J23 CAN 3V3_{EN}, J24 CAN UP_{EN}, J25 CAN Downstream, J26 Use DB9 VBUS, J27 DE9_Socket_MountingHoles, SW3 CAN Termination Select, U10 MCP2542FD-E/SN

Commit message: Finalized schematic diagram. Only needs formatting fixes and resistor component sourcing info
Parts:
- renumbered J17 to J20, J18 to J21, J19 to J22, J20 to J23, J21 to J24, J22 to J25, J23 to J26, J24 to J27, J25 to J28, J26 to J29, J27 to J30, TP19 to TP22, TP20 to TP23, TP21 to TP24
Changed lines of the file:
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@@
 		(on_board yes)
 		(dnp no)
-		(property "Reference" "J25"
+		(property "Reference" "J28"
 			(at 235.712 77.47 0)
 			(effects
@@
 			(project "LiF_FC-PCB_rev1"
 				(path "/9e3e8da7-e506-46c9-90e5-307e4ad30d29/77827f91-166d-41e9-a525-15815c2a0550"
-					(reference "J25")
+					(reference "J28")
 					(unit 1)
 				)
@@
 		(on_board yes)
 		(dnp no)
-		(property "Reference" "#PWR057"
+		(property "Reference" "#PWR060"
 			(at 223.52 78.74 0)
 			(effects
@@
 			(project "LiF_FC-PCB_rev1"
 				(path "/9e3e8da7-e506-46c9-90e5-307e4ad30d29/77827f91-166d-41e9-a525-15815c2a0550"
-					(reference "#PWR057")
+					(reference "#PWR060")
 					(unit 1)
 				)
@@
 		(on_board yes)
 		(dnp no)
-		(property "Reference" "#PWR062"
+		(property "Reference" "#PWR065"
 			(at 76.2 146.05 0)
 			(effects
@@
 			(project "LiF_FC-PCB_rev1"
 				(path "/9e3e8da7-e506-46c9-90e5-307e4ad30d29/77827f91-166d-41e9-a525-15815c2a0550"
-					(reference "#PWR062")
+					(reference "#PWR065")
 					(unit 1)
 				)
@@
 		(on_board yes)
 		(dnp no)
-		(property "Reference" "#PWR059"
+		(property "Reference" "#PWR062"
 			(at 223.52 120.65 0)
 			(effects
@@
 			(project "LiF_FC-PCB_rev1"
 				(path "/9e3e8da7-e506-46c9-90e5-307e4ad30d29/77827f91-166d-41e9-a525-15815c2a0550"
-					(reference "#PWR059")
+					(reference "#PWR062")
 					(unit 1)
 				)
@@
 		(on_board yes)
 		(dnp no)
-		(property "Reference" "J26"
+		(property "Reference" "J29"
 			(at 119.888 95.504 90)
 			(effects
@@
 			(project "LiF_FC-PCB_rev1"
 				(path "/9e3e8da7-e506-46c9-90e5-307e4ad30d29/77827f91-166d-41e9-a525-15815c2a0550"
-					(reference "J26")
+					(reference "J29")
 					(unit 1)
 				)
@@
 		(on_board yes)
 		(dnp no)
-		(property "Reference" "TP21"
+		(property "Reference" "TP24"
 			(at 142.748 132.588 0)
 			(effects
@@
 			(project "LiF_FC-PCB_rev1"
 				(path "/9e3e8da7-e506-46c9-90e5-307e4ad30d29/77827f91-166d-41e9-a525-15815c2a0550"
-					(reference "TP21")
+					(reference "TP24")
 					(unit 1)
 				)
@@
 		(on_board yes)
 		(dnp no)
-		(property "Reference" "#PWR065"
+		(property "Reference" "#PWR068"
 			(at 54.61 179.07 0)
 			(effects
@@
 			(project "LiF_FC-PCB_rev1"
 				(path "/9e3e8da7-e506-46c9-90e5-307e4ad30d29/77827f91-166d-41e9-a525-15815c2a0550"
-					(reference "#PWR065")
+					(reference "#PWR068")
 					(unit 1)
 				)
@@
 		(on_board yes)
 		(dnp no)
-		(property "Reference" "J20"
+		(property "Reference" "J23"
 			(at 57.912 54.864 90)
 			(effects
@@
 			(project "LiF_FC-PCB_rev1"
 				(path "/9e3e8da7-e506-46c9-90e5-307e4ad30d29/77827f91-166d-41e9-a525-15815c2a0550"
-					(reference "J20")
+					(reference "J23")
 					(unit 1)
 				)
@@
 		(dnp no)
 		(fields_autoplaced yes)
-		(property "Reference" "J27"
+		(property "Reference" "J30"
 			(at 240.03 139.6999 0)
 			(effects
@@
 			(project ""
 				(path "/9e3e8da7-e506-46c9-90e5-307e4ad30d29/77827f91-166d-41e9-a525-15815c2a0550"
-					(reference "J27")
+					(reference "J30")
 					(unit 1)
 				)
@@
 		(on_board yes)
 		(dnp no)
-		(property "Reference" "#PWR056"
+		(property "Reference" "#PWR059"
 			(at 190.5 67.31 0)
 			(effects
@@
 			(project "LiF_FC-PCB_rev1"
 				(path "/9e3e8da7-e506-46c9-90e5-307e4ad30d29/77827f91-166d-41e9-a525-15815c2a0550"
-					(reference "#PWR056")
+					(reference "#PWR059")
 					(unit 1)
 				)
@@
 		(on_board yes)
 		(dnp no)
-		(property "Reference" "TP20"
+		(property "Reference" "TP23"
 			(at 132.588 132.588 0)
 			(effects
@@
 			(project "LiF_FC-PCB_rev1"
 				(path "/9e3e8da7-e506-46c9-90e5-307e4ad30d29/77827f91-166d-41e9-a525-15815c2a0550"
-					(reference "TP20")
+					(reference "TP23")
 					(unit 1)
 				)
@@
 		(on_board yes)
 		(dnp no)
-		(property "Reference" "#PWR063"
+		(property "Reference" "#PWR066"
 			(at 223.52 163.83 0)
 			(effects
@@
 			(project "LiF_FC-PCB_rev1"
 				(path "/9e3e8da7-e506-46c9-90e5-307e4ad30d29/77827f91-166d-41e9-a525-15815c2a0550"
-					(reference "#PWR063")
+					(reference "#PWR066")
 					(unit 1)
 				)
@@
 		(on_board yes)
 		(dnp no)
-		(property "Reference" "#PWR058"
+		(property "Reference" "#PWR061"
 			(at 190.5 109.22 0)
 			(effects
@@
 			(project "LiF_FC-PCB_rev1"
 				(path "/9e3e8da7-e506-46c9-90e5-307e4ad30d29/77827f91-166d-41e9-a525-15815c2a0550"
-					(reference "#PWR058")
+					(reference "#PWR061")
 					(unit 1)
 				)
@@
 		(on_board yes)
 		(dnp no)
-		(property "Reference" "J17"
+		(property "Reference" "J20"
 			(at 254.762 25.654 90)
 			(effects
@@
 			(project "LiF_FC-PCB_rev1"
 				(path "/9e3e8da7-e506-46c9-90e5-307e4ad30d29/77827f91-166d-41e9-a525-15815c2a0550"
-					(reference "J17")
+					(reference "J20")
 					(unit 1)
 				)
@@
 		(on_board yes)
 		(dnp no)
-		(property "Reference" "J23"
+		(property "Reference" "J26"
 			(at 57.912 73.914 90)
 			(effects
@@
 			(project "LiF_FC-PCB_rev1"
 				(path "/9e3e8da7-e506-46c9-90e5-307e4ad30d29/77827f91-166d-41e9-a525-15815c2a0550"
-					(reference "J23")
+					(reference "J26")
 					(unit 1)
 				)
@@
 		(on_board yes)
 		(dnp no)
-		(property "Reference" "J24"
+		(property "Reference" "J27"
 			(at 123.952 75.184 90)
 			(effects
@@
 			(project "LiF_FC-PCB_rev1"
 				(path "/9e3e8da7-e506-46c9-90e5-307e4ad30d29/77827f91-166d-41e9-a525-15815c2a0550"
-					(reference "J24")
+					(reference "J27")
 					(unit 1)
 				)
@@
 		(on_board yes)
 		(dnp no)
-		(property "Reference" "#PWR060"
+		(property "Reference" "#PWR063"
 			(at 140.97 144.78 0)
 			(effects
@@
 			(project "LiF_FC-PCB_rev1"
 				(path "/9e3e8da7-e506-46c9-90e5-307e4ad30d29/77827f91-166d-41e9-a525-15815c2a0550"
-					(reference "#PWR060")
+					(reference "#PWR063")
 					(unit 1)
 				)
@@
 		(on_board yes)
 		(dnp no)
-		(property "Reference" "J18"
+		(property "Reference" "J21"
 			(at 123.952 37.084 90)
 			(effects
@@
 			(project "LiF_FC-PCB_rev1"
 				(path "/9e3e8da7-e506-46c9-90e5-307e4ad30d29/77827f91-166d-41e9-a525-15815c2a0550"
-					(reference "J18")
+					(reference "J21")
 					(unit 1)
 				)
@@
 		(on_board yes)
 		(dnp no)
-		(property "Reference" "#PWR061"
+		(property "Reference" "#PWR064"
 			(at 66.04 146.05 0)
 			(effects
@@
 			(project "LiF_FC-PCB_rev1"
 				(path "/9e3e8da7-e506-46c9-90e5-307e4ad30d29/77827f91-166d-41e9-a525-15815c2a0550"
-					(reference "#PWR061")
+					(reference "#PWR064")
 					(unit 1)
 				)
@@
 		(on_board yes)
 		(dnp no)
-		(property "Reference" "#PWR066"
+		(property "Reference" "#PWR069"
 			(at 72.39 179.07 0)
 			(effects
@@
 			(project "LiF_FC-PCB_rev1"
 				(path "/9e3e8da7-e506-46c9-90e5-307e4ad30d29/77827f91-166d-41e9-a525-15815c2a0550"
-					(reference "#PWR066")
+					(reference "#PWR069")
 					(unit 1)
 				)
@@
 		(on_board yes)
 		(dnp no)
-		(property "Reference" "TP19"
+		(property "Reference" "TP22"
 			(at 123.952 132.588 0)
 			(effects
@@
 			(project "LiF_FC-PCB_rev1"
 				(path "/9e3e8da7-e506-46c9-90e5-307e4ad30d29/77827f91-166d-41e9-a525-15815c2a0550"
-					(reference "TP19")
+					(reference "TP22")
 					(unit 1)
 				)
@@
 		(on_board yes)
 		(dnp no)
-		(property "Reference" "J22"
+		(property "Reference" "J25"
 			(at 254.762 67.564 90)
 			(effects
@@
 			(project "LiF_FC-PCB_rev1"
 				(path "/9e3e8da7-e506-46c9-90e5-307e4ad30d29/77827f91-166d-41e9-a525-15815c2a0550"
-					(reference "J22")
+					(reference "J25")
 					(unit 1)
 				)
@@
 		(on_board yes)
 		(dnp no)
-		(property "Reference" "#PWR064"
+		(property "Reference" "#PWR067"
 			(at 234.95 163.83 0)
 			(effects
@@
 			(project "LiF_FC-PCB_rev1"
 				(path "/9e3e8da7-e506-46c9-90e5-307e4ad30d29/77827f91-166d-41e9-a525-15815c2a0550"
-					(reference "#PWR064")
+					(reference "#PWR067")
 					(unit 1)
 				)
@@
 		(on_board yes)
 		(dnp no)
-		(property "Reference" "J19"
+		(property "Reference" "J22"
 			(at 236.982 34.798 0)
 			(effects
@@
 			(project "LiF_FC-PCB_rev1"
 				(path "/9e3e8da7-e506-46c9-90e5-307e4ad30d29/77827f91-166d-41e9-a525-15815c2a0550"
-					(reference "J19")
+					(reference "J22")
 					(unit 1)
 				)
@@
 		(on_board yes)
 		(dnp no)
-		(property "Reference" "J21"
+		(property "Reference" "J24"
 			(at 119.888 56.134 90)
 			(effects
@@
 			(project "LiF_FC-PCB_rev1"
 				(path "/9e3e8da7-e506-46c9-90e5-307e4ad30d29/77827f91-166d-41e9-a525-15815c2a0550"
-					(reference "J21")
+					(reference "J24")
 					(unit 1)
 				)
@@
 		(on_board yes)
 		(dnp no)
-		(property "Reference" "#PWR067"
+		(property "Reference" "#PWR070"
 			(at 128.27 180.34 0)
 			(effects
@@
 			(project "LiF_FC-PCB_rev1"
 				(path "/9e3e8da7-e506-46c9-90e5-307e4ad30d29/77827f91-166d-41e9-a525-15815c2a0550"
-					(reference "#PWR067")
+					(reference "#PWR070")
 					(unit 1)
 				)

Commit message: set up board configuration and started routing PCB
Parts:
- TP22, TP23, TP24: footprint TestPoint:TestPoint_Bridge_Pitch2.54mm_Drill1.0mm -> TestPoint:TestPoint_Loop_D1.80mm_Drill1.0mm_Beaded
Connections:
- net CANH renamed CAN+
- net CANL renamed CAN-
Changed lines of the file:
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@@
 		)
 	)
-	(label "CANL"
+	(label "CAN-"
 		(at 92.71 158.75 180)
 		(effects
@@
 		)
 	)
-	(label "CANL"
+	(label "CAN-"
 		(at 252.73 100.33 180)
 		(effects
@@
 		)
 	)
-	(label "CANH"
+	(label "CAN+"
 		(at 92.71 153.67 180)
 		(effects
@@
 		)
 	)
-	(label "CANH"
+	(label "CAN+"
 		(at 212.09 138.43 0)
 		(effects
@@
 		)
 	)
-	(label "CANH"
+	(label "CAN+"
 		(at 252.73 52.07 180)
 		(effects
@@
 		)
 	)
-	(label "CANH"
+	(label "CAN+"
 		(at 252.73 93.98 180)
 		(effects
@@
 		)
 	)
-	(label "CANL"
+	(label "CAN-"
 		(at 252.73 58.42 180)
 		(effects
@@
 		)
 	)
-	(label "CANL"
+	(label "CAN-"
 		(at 212.09 135.89 0)
 		(effects
@@
 			)
 		)
-		(property "Footprint" "TestPoint:TestPoint_Bridge_Pitch2.54mm_Drill1.0mm"
+		(property "Footprint" "TestPoint:TestPoint_Loop_D1.80mm_Drill1.0mm_Beaded"
 			(at 146.05 137.16 0)
 			(effects
@@
 			)
 		)
-		(property "Footprint" "TestPoint:TestPoint_Bridge_Pitch2.54mm_Drill1.0mm"
+		(property "Footprint" "TestPoint:TestPoint_Loop_D1.80mm_Drill1.0mm_Beaded"
 			(at 135.89 137.16 0)
 			(effects
@@
 			)
 		)
-		(property "Footprint" "TestPoint:TestPoint_Bridge_Pitch2.54mm_Drill1.0mm"
+		(property "Footprint" "TestPoint:TestPoint_Loop_D1.80mm_Drill1.0mm_Beaded"
 			(at 120.65 137.16 0)
 			(effects

Commit message: backup before expanding the board size
Parts:
- removed SW3: CAN Termination Select, LiF_PCB_Footprints:SW_SLW-883935-2A-D, symbol Switch:SW_SPDT
- added J44: CAN, Connector_JST:JST_PH_B4B-PH-K_1x04_P2.00mm_Vertical, symbol Connector_Generic:Conn_01x04
- added SW3: CAN Termination, LiF_PCB_Footprints:SW_JS202011JCQN, symbol Switch:SW_DPDT_x2
- J30: now not fitted; now left out of the parts list
Connections:
- net CAN+: now also J44.2 (Pin_2), SW3.5 (B)
- net CAN-: now also J44.1 (Pin_1)
- net GND: now also J44.3 (Pin_3)
- net VBUS_DB9: now also J44.4 (Pin_4)
- net at R53.2: now also SW3.6 (C)
- no-connect marks 10 -> 13
Other:
- note added: "Aux CAN Connectors"
- note removed: "DB-9 CAN Connector"

Commit message: backup before leaving school
Parts:
- J20, J21, J23, J24, J25, J26, J27, J29: footprint Connector_PinHeader_2.54mm:PinHeader_1x02_P2.54mm_Vertical -> Connector_PinHeader_2.54mm:PinHeader_1x02_P2.54mm_Vertical_SMD_Pin1Left
Changed lines of the file:
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@@
 			)
 		)
-		(property "Footprint" "Connector_PinHeader_2.54mm:PinHeader_1x02_P2.54mm_Vertical"
+		(property "Footprint" "Connector_PinHeader_2.54mm:PinHeader_1x02_P2.54mm_Vertical_SMD_Pin1Left"
 			(at 120.65 96.52 0)
 			(effects
@@
 			)
 		)
-		(property "Footprint" "Connector_PinHeader_2.54mm:PinHeader_1x02_P2.54mm_Vertical"
+		(property "Footprint" "Connector_PinHeader_2.54mm:PinHeader_1x02_P2.54mm_Vertical_SMD_Pin1Left"
 			(at 57.15 55.88 0)
 			(effects
@@
 			)
 		)
-		(property "Footprint" "Connector_PinHeader_2.54mm:PinHeader_1x02_P2.54mm_Vertical"
+		(property "Footprint" "Connector_PinHeader_2.54mm:PinHeader_1x02_P2.54mm_Vertical_SMD_Pin1Left"
 			(at 254 26.67 0)
 			(effects
@@
 			)
 		)
-		(property "Footprint" "Connector_PinHeader_2.54mm:PinHeader_1x02_P2.54mm_Vertical"
+		(property "Footprint" "Connector_PinHeader_2.54mm:PinHeader_1x02_P2.54mm_Vertical_SMD_Pin1Left"
 			(at 57.15 74.93 0)
 			(effects
@@
 			)
 		)
-		(property "Footprint" "Connector_PinHeader_2.54mm:PinHeader_1x02_P2.54mm_Vertical"
+		(property "Footprint" "Connector_PinHeader_2.54mm:PinHeader_1x02_P2.54mm_Vertical_SMD_Pin1Left"
 			(at 123.19 76.2 0)
 			(effects
@@
 			)
 		)
-		(property "Footprint" "Connector_PinHeader_2.54mm:PinHeader_1x02_P2.54mm_Vertical"
+		(property "Footprint" "Connector_PinHeader_2.54mm:PinHeader_1x02_P2.54mm_Vertical_SMD_Pin1Left"
 			(at 123.19 38.1 0)
 			(effects
@@
 			)
 		)
-		(property "Footprint" "Connector_PinHeader_2.54mm:PinHeader_1x02_P2.54mm_Vertical"
+		(property "Footprint" "Connector_PinHeader_2.54mm:PinHeader_1x02_P2.54mm_Vertical_SMD_Pin1Left"
 			(at 254 68.58 0)
 			(effects
@@
 			)
 		)
-		(property "Footprint" "Connector_PinHeader_2.54mm:PinHeader_1x02_P2.54mm_Vertical"
+		(property "Footprint" "Connector_PinHeader_2.54mm:PinHeader_1x02_P2.54mm_Vertical_SMD_Pin1Left"
 			(at 120.65 57.15 0)
 			(effects
