File: KiCAD/LiF_FC-PCB_rev1/LiF_LoadCell.kicad_sch (KiCad schematic)
At the start: 20 parts, among them J10 LC 3V3_{EN}, J11 Load Cell, J12 LC 5V0_{EN}, U5 MCP6N11-xxxE/SN, U8 NCV8114ASN165T1G

Commit message: reverted 5V reg, reworked power distribution logic, swapped power OR-ing ICs
Parts:
- added C11: 1u, Capacitor_SMD:C_0805_2012Metric, symbol Device:C
- added C12: 0.1u, Capacitor_SMD:C_0805_2012Metric, symbol Device:C
Connections:
- net E+: now also C11.1, C12.1
- net GND renamed GNDA
- net GNDA: now also C11.2, C12.2
Other:
- moved on the sheet: J11

Commit message: Finished schematics, mostly. Only MCU sheet left. Doing component sourcing
Parts:
- C25: DKPN (none) -> 490-12005-1-ND; PN (none) -> GRM21BR72A104KAC4L
- C26: renamed from C28; DKPN (none) -> 490-12005-1-ND; PN (none) -> GRM21BR72A104KAC4L
- C27: renamed from C30; DKPN (none) -> 490-12005-1-ND; PN (none) -> GRM21BR72A104KAC4L
- C28: renamed from C11; DKPN (none) -> 490-1691-1-ND; PN (none) -> GRM21BR71C105KA01L
- C29: renamed from C12; DKPN (none) -> 490-12005-1-ND; PN (none) -> GRM21BR72A104KAC4L
- C30: renamed from C29; DKPN (none) -> 490-1691-1-ND; PN (none) -> GRM21BR71C105KA01L
- C31: renamed from C26; DKPN (none) -> 490-1691-1-ND; PN (none) -> GRM21BR71C105KA01L
- C32: renamed from C27; DKPN (none) -> 490-12005-1-ND; PN (none) -> GRM21BR72A104KAC4L
- J13: renamed from J12; footprint Connector_PinHeader_1.27mm:PinHeader_1x02_P1.27mm_Vertical -> Connector_PinHeader_2.54mm:PinHeader_1x02_P2.54mm_Vertical
- J14: renamed from J10; footprint Connector_PinHeader_1.27mm:PinHeader_1x02_P1.27mm_Vertical -> Connector_PinHeader_2.54mm:PinHeader_1x02_P2.54mm_Vertical
- renumbered J11 to J15, R29 to R33, R36 to R34, R37 to R35, R35 to R36, R30 to R37, R31 to R38, R34 to R39, R33 to R40, R32 to R41, U5 to U8, U8 to U9
Other:
- note added: "Lithium Firefly - Load Cell Signal Conditioning"
- note removed: "LiF - Load Cell Signal Conditioning Circuit"
- company: (none) -> Lithium Firefly Team

Commit message: fixing ERC bugs on schematic. Only MCU left
Parts:
- added TP19: V^{-}, TestPoint:TestPoint_Bridge_Pitch2.54mm_Drill1.0mm, symbol Connector:TestPoint
- added TP20: V^{+}, TestPoint:TestPoint_Bridge_Pitch2.54mm_Drill1.0mm, symbol Connector:TestPoint
- added TP21: LC, TestPoint:TestPoint_Bridge_Pitch2.54mm_Drill1.0mm, symbol Connector:TestPoint
- added TP22: FLT, TestPoint:TestPoint_Bridge_Pitch2.54mm_Drill1.0mm, symbol Connector:TestPoint
- added TP23: V_{REF}, TestPoint:TestPoint_Bridge_Pitch2.54mm_Drill1.0mm, symbol Connector:TestPoint
- added TP24, TP25: GND, TestPoint:TestPoint_Bridge_Pitch2.54mm_Drill1.0mm, symbol Connector:TestPoint
- U9: DKPN (none) -> 488-NCV8114ASN165T1GCT-ND; PN (none) -> NCV8114ASN165T1G
Connections:
- net GNDA: now also TP24.1, TP25.1
- net LC V_{OUT}: now also TP22.1
- net MCP V_{OUT}: now also TP21.1
- net V_{REF}: now also TP23.1
- net at C26.1, R33.1, U8.2 (V^{-}): now also TP19.1
- net at C26.2, R37.2, U8.3 (V^{+}): now also TP20.1

Commit message: Added MCU pinout, shanged shift registers to GPIO expanders to save pins on MCU
Parts:
- renumbered J13 to J14, J14 to J15, J15 to J16, R33 to R34, R34 to R35, R35 to R36, R36 to R37, R37 to R38, R38 to R39, R39 to R40, R40 to R41, R41 to R42, TP19 to TP12, TP25 to TP13, TP21 to TP14, TP22 to TP15, TP20 to TP16, TP24 to TP17, TP23 to TP18
Other:
- title: (none) -> Lithium Firefly Custom FC/CC PCB
Changed lines of the file:
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@@
 	(paper "A4")
 	(title_block
+		(title "Lithium Firefly Custom FC/CC PCB")
+		(date "2026-07-11")
 		(rev "1")
 		(company "Lithium Firefly Team")
+		(comment 1 "Designed by RY and MR")
 		(comment 2 "Verified by MR")
 	)
@@
 		(on_board yes)
 		(dnp no)
-		(property "Reference" "TP19"
+		(property "Reference" "TP12"
 			(at 137.668 57.658 0)
 			(effects
@@
 			(project "LiF_FC-PCB_rev1"
 				(path "/9e3e8da7-e506-46c9-90e5-307e4ad30d29/17577359-df8d-4d28-9071-787d31b1b6da"
-					(reference "TP19")
+					(reference "TP12")
 					(unit 1)
 				)
@@
 		(on_board yes)
 		(dnp yes)
-		(property "Reference" "R34"
+		(property "Reference" "R35"
 			(at 53.34 68.58 90)
 			(effects
@@
 			(project "LiF_FC-PCB_rev1"
 				(path "/9e3e8da7-e506-46c9-90e5-307e4ad30d29/17577359-df8d-4d28-9071-787d31b1b6da"
-					(reference "R34")
+					(reference "R35")
 					(unit 1)
 				)
@@
 		(on_board yes)
 		(dnp no)
-		(property "Reference" "TP25"
+		(property "Reference" "TP13"
 			(at 206.248 57.658 0)
 			(effects
@@
 			(project "LiF_FC-PCB_rev1"
 				(path "/9e3e8da7-e506-46c9-90e5-307e4ad30d29/17577359-df8d-4d28-9071-787d31b1b6da"
-					(reference "TP25")
+					(reference "TP13")
 					(unit 1)
 				)
@@
 		(on_board yes)
 		(dnp no)
-		(property "Reference" "#PWR0116"
+		(property "Reference" "#PWR048"
 			(at 176.53 127 0)
 			(effects
@@
 			(project "LiF_FC-PCB_rev1"
 				(path "/9e3e8da7-e506-46c9-90e5-307e4ad30d29/17577359-df8d-4d28-9071-787d31b1b6da"
-					(reference "#PWR0116")
+					(reference "#PWR048")
 					(unit 1)
 				)
@@
 		(on_board yes)
 		(dnp no)
-		(property "Reference" "TP22"
+		(property "Reference" "TP15"
 			(at 271.018 60.198 0)
 			(effects
@@
 			(project "LiF_FC-PCB_rev1"
 				(path "/9e3e8da7-e506-46c9-90e5-307e4ad30d29/17577359-df8d-4d28-9071-787d31b1b6da"
-					(reference "TP22")
+					(reference "TP15")
 					(unit 1)
 				)
@@
 		(on_board yes)
 		(dnp no)
-		(property "Reference" "#PWR047"
+		(property "Reference" "#PWR046"
 			(at 256.54 91.44 0)
 			(effects
@@
 			(project "LiF_FC-PCB_rev1"
 				(path "/9e3e8da7-e506-46c9-90e5-307e4ad30d29/17577359-df8d-4d28-9071-787d31b1b6da"
-					(reference "#PWR047")
+					(reference "#PWR046")
 					(unit 1)
 				)
@@
 		(on_board yes)
 		(dnp no)
-		(property "Reference" "TP24"
+		(property "Reference" "TP17"
 			(at 178.308 114.808 0)
 			(effects
@@
 			(project "LiF_FC-PCB_rev1"
 				(path "/9e3e8da7-e506-46c9-90e5-307e4ad30d29/17577359-df8d-4d28-9071-787d31b1b6da"
-					(reference "TP24")
+					(reference "TP17")
 					(unit 1)
 				)
@@
 		(on_board yes)
 		(dnp yes)
-		(property "Reference" "R38"
+		(property "Reference" "R39"
 			(at 53.34 85.09 90)
 			(effects
@@
 			(project "LiF_FC-PCB_rev1"
 				(path "/9e3e8da7-e506-46c9-90e5-307e4ad30d29/17577359-df8d-4d28-9071-787d31b1b6da"
-					(reference "R38")
+					(reference "R39")
 					(unit 1)
 				)
@@
 		(dnp no)
 		(fields_autoplaced yes)
-		(property "Reference" "R35"
+		(property "Reference" "R36"
 			(at 246.38 63.5 90)
 			(effects
@@
 			(project "LiF_FC-PCB_rev1"
 				(path "/9e3e8da7-e506-46c9-90e5-307e4ad30d29/17577359-df8d-4d28-9071-787d31b1b6da"
-					(reference "R35")
+					(reference "R36")
 					(unit 1)
 				)
@@
 		(dnp no)
 		(fields_autoplaced yes)
-		(property "Reference" "R36"
+		(property "Reference" "R37"
 			(at 179.07 76.1999 0)
 			(effects
@@
 			(project "LiF_FC-PCB_rev1"
 				(path "/9e3e8da7-e506-46c9-90e5-307e4ad30d29/17577359-df8d-4d28-9071-787d31b1b6da"
-					(reference "R36")
+					(reference "R37")
 					(unit 1)
 				)
@@
 		(on_board yes)
 		(dnp no)
-		(property "Reference" "TP21"
+		(property "Reference" "TP14"
 			(at 197.612 60.198 0)
 			(effects
@@
 			(project "LiF_FC-PCB_rev1"
 				(path "/9e3e8da7-e506-46c9-90e5-307e4ad30d29/17577359-df8d-4d28-9071-787d31b1b6da"
-					(reference "TP21")
+					(reference "TP14")
 					(unit 1)
 				)
@@
 		(on_board yes)
 		(dnp no)
-		(property "Reference" "#PWR0117"
+		(property "Reference" "#PWR045"
 			(at 204.47 69.85 0)
 			(effects
@@
 			(project "LiF_FC-PCB_rev1"
 				(path "/9e3e8da7-e506-46c9-90e5-307e4ad30d29/17577359-df8d-4d28-9071-787d31b1b6da"
-					(reference "#PWR0117")
+					(reference "#PWR045")
 					(unit 1)
 				)
@@
 		(dnp no)
 		(fields_autoplaced yes)
-		(property "Reference" "R41"
+		(property "Reference" "R42"
 			(at 171.45 138.4299 0)
 			(effects
@@
 			(project "LiF_FC-PCB_rev1"
 				(path "/9e3e8da7-e506-46c9-90e5-307e4ad30d29/17577359-df8d-4d28-9071-787d31b1b6da"
-					(reference "R41")
+					(reference "R42")
 					(unit 1)
 				)
@@
 		(on_board yes)
 		(dnp no)
-		(property "Reference" "J14"
+		(property "Reference" "J15"
 			(at 55.372 72.644 90)
 			(effects
@@
 			(project "LiF_FC-PCB_rev1"
 				(path "/9e3e8da7-e506-46c9-90e5-307e4ad30d29/17577359-df8d-4d28-9071-787d31b1b6da"
-					(reference "J14")
+					(reference "J15")
 					(unit 1)
 				)
@@
 		(on_board yes)
 		(dnp no)
-		(property "Reference" "TP23"
+		(property "Reference" "TP18"
 			(at 156.972 121.158 0)
 			(effects
@@
 			(project "LiF_FC-PCB_rev1"
 				(path "/9e3e8da7-e506-46c9-90e5-307e4ad30d29/17577359-df8d-4d28-9071-787d31b1b6da"
-					(reference "TP23")
+					(reference "TP18")
 					(unit 1)
 				)
@@
 		(on_board yes)
 		(dnp no)
-		(property "Reference" "TP20"
+		(property "Reference" "TP16"
 			(at 137.668 87.122 0)
 			(effects
@@
 			(project "LiF_FC-PCB_rev1"
 				(path "/9e3e8da7-e506-46c9-90e5-307e4ad30d29/17577359-df8d-4d28-9071-787d31b1b6da"
-					(reference "TP20")
+					(reference "TP16")
 					(unit 1)
 				)
@@
 		(dnp no)
 		(fields_autoplaced yes)
-		(property "Reference" "R33"
+		(property "Reference" "R34"
 			(at 120.65 57.15 90)
 			(effects
@@
 			(project "LiF_FC-PCB_rev1"
 				(path "/9e3e8da7-e506-46c9-90e5-307e4ad30d29/17577359-df8d-4d28-9071-787d31b1b6da"
-					(reference "R33")
+					(reference "R34")
 					(unit 1)
 				)
@@
 		(dnp no)
 		(fields_autoplaced yes)
-		(property "Reference" "R40"
+		(property "Reference" "R41"
 			(at 179.07 95.2499 0)
 			(effects
@@
 			(project "LiF_FC-PCB_rev1"
 				(path "/9e3e8da7-e506-46c9-90e5-307e4ad30d29/17577359-df8d-4d28-9071-787d31b1b6da"
-					(reference "R40")
+					(reference "R41")
 					(unit 1)
 				)
@@
 		(on_board yes)
 		(dnp no)
-		(property "Reference" "J13"
+		(property "Reference" "J14"
 			(at 55.372 56.134 90)
 			(effects
@@
 			(project "LiF_FC-PCB_rev1"
 				(path "/9e3e8da7-e506-46c9-90e5-307e4ad30d29/17577359-df8d-4d28-9071-787d31b1b6da"
-					(reference "J13")
+					(reference "J14")
 					(unit 1)
 				)
@@
 		(on_board yes)
 		(dnp no)
-		(property "Reference" "#PWR046"
+		(property "Reference" "#PWR044"
 			(at 147.32 63.5 0)
 			(effects
@@
 			(project "LiF_FC-PCB_rev1"
 				(path "/9e3e8da7-e506-46c9-90e5-307e4ad30d29/17577359-df8d-4d28-9071-787d31b1b6da"
-					(reference "#PWR046")
+					(reference "#PWR044")
 					(unit 1)
 				)
@@
 		(on_board yes)
 		(dnp no)
-		(property "Reference" "#PWR048"
+		(property "Reference" "#PWR047"
 			(at 153.67 95.25 0)
 			(effects
@@
 			(project "LiF_FC-PCB_rev1"
 				(path "/9e3e8da7-e506-46c9-90e5-307e4ad30d29/17577359-df8d-4d28-9071-787d31b1b6da"
-					(reference "#PWR048")
+					(reference "#PWR047")
 					(unit 1)
 				)
@@
 		(dnp no)
 		(fields_autoplaced yes)
-		(property "Reference" "R39"
+		(property "Reference" "R40"
 			(at 179.07 85.0899 0)
 			(effects
@@
 			(project "LiF_FC-PCB_rev1"
 				(path "/9e3e8da7-e506-46c9-90e5-307e4ad30d29/17577359-df8d-4d28-9071-787d31b1b6da"
-					(reference "R39")
+					(reference "R40")
 					(unit 1)
 				)
@@
 		(on_board yes)
 		(dnp no)
-		(property "Reference" "J15"
+		(property "Reference" "J16"
 			(at 22.86 121.92 0)
 			(effects
@@
 			(project ""
 				(path "/9e3e8da7-e506-46c9-90e5-307e4ad30d29/17577359-df8d-4d28-9071-787d31b1b6da"
-					(reference "J15")
+					(reference "J16")
 					(unit 1)
 				)
@@
 		(on_board yes)
 		(dnp no)
-		(property "Reference" "R37"
+		(property "Reference" "R38"
 			(at 120.65 82.55 90)
 			(effects
@@
 			(project "LiF_FC-PCB_rev1"
 				(path "/9e3e8da7-e506-46c9-90e5-307e4ad30d29/17577359-df8d-4d28-9071-787d31b1b6da"
-					(reference "R37")
+					(reference "R38")
 					(unit 1)
 				)

Commit message: Finalized schematic diagram. Only needs formatting fixes and resistor component sourcing info
Parts:
- renumbered J14 to J17, J15 to J18, J16 to J19, TP12 to TP15, TP13 to TP16, TP14 to TP17, TP15 to TP18, TP16 to TP19, TP17 to TP20, TP18 to TP21
Changed lines of the file:
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@@
 		(on_board yes)
 		(dnp no)
-		(property "Reference" "TP12"
+		(property "Reference" "TP15"
 			(at 137.668 57.658 0)
 			(effects
@@
 			(project "LiF_FC-PCB_rev1"
 				(path "/9e3e8da7-e506-46c9-90e5-307e4ad30d29/17577359-df8d-4d28-9071-787d31b1b6da"
-					(reference "TP12")
+					(reference "TP15")
 					(unit 1)
 				)
@@
 		(on_board yes)
 		(dnp no)
-		(property "Reference" "TP13"
+		(property "Reference" "TP16"
 			(at 206.248 57.658 0)
 			(effects
@@
 			(project "LiF_FC-PCB_rev1"
 				(path "/9e3e8da7-e506-46c9-90e5-307e4ad30d29/17577359-df8d-4d28-9071-787d31b1b6da"
-					(reference "TP13")
+					(reference "TP16")
 					(unit 1)
 				)
@@
 		(on_board yes)
 		(dnp no)
-		(property "Reference" "#PWR048"
+		(property "Reference" "#PWR051"
 			(at 176.53 127 0)
 			(effects
@@
 			(project "LiF_FC-PCB_rev1"
 				(path "/9e3e8da7-e506-46c9-90e5-307e4ad30d29/17577359-df8d-4d28-9071-787d31b1b6da"
-					(reference "#PWR048")
+					(reference "#PWR051")
 					(unit 1)
 				)
@@
 		(on_board yes)
 		(dnp no)
-		(property "Reference" "TP15"
+		(property "Reference" "TP18"
 			(at 271.018 60.198 0)
 			(effects
@@
 			(project "LiF_FC-PCB_rev1"
 				(path "/9e3e8da7-e506-46c9-90e5-307e4ad30d29/17577359-df8d-4d28-9071-787d31b1b6da"
-					(reference "TP15")
+					(reference "TP18")
 					(unit 1)
 				)
@@
 		(on_board yes)
 		(dnp no)
-		(property "Reference" "#PWR046"
+		(property "Reference" "#PWR049"
 			(at 256.54 91.44 0)
 			(effects
@@
 			(project "LiF_FC-PCB_rev1"
 				(path "/9e3e8da7-e506-46c9-90e5-307e4ad30d29/17577359-df8d-4d28-9071-787d31b1b6da"
-					(reference "#PWR046")
+					(reference "#PWR049")
 					(unit 1)
 				)
@@
 		(on_board yes)
 		(dnp no)
-		(property "Reference" "TP17"
+		(property "Reference" "TP20"
 			(at 178.308 114.808 0)
 			(effects
@@
 			(project "LiF_FC-PCB_rev1"
 				(path "/9e3e8da7-e506-46c9-90e5-307e4ad30d29/17577359-df8d-4d28-9071-787d31b1b6da"
-					(reference "TP17")
+					(reference "TP20")
 					(unit 1)
 				)
@@
 		(on_board yes)
 		(dnp no)
-		(property "Reference" "TP14"
+		(property "Reference" "TP17"
 			(at 197.612 60.198 0)
 			(effects
@@
 			(project "LiF_FC-PCB_rev1"
 				(path "/9e3e8da7-e506-46c9-90e5-307e4ad30d29/17577359-df8d-4d28-9071-787d31b1b6da"
-					(reference "TP14")
+					(reference "TP17")
 					(unit 1)
 				)
@@
 		(on_board yes)
 		(dnp no)
-		(property "Reference" "#PWR045"
+		(property "Reference" "#PWR048"
 			(at 204.47 69.85 0)
 			(effects
@@
 			(project "LiF_FC-PCB_rev1"
 				(path "/9e3e8da7-e506-46c9-90e5-307e4ad30d29/17577359-df8d-4d28-9071-787d31b1b6da"
-					(reference "#PWR045")
+					(reference "#PWR048")
 					(unit 1)
 				)
@@
 		(on_board yes)
 		(dnp no)
-		(property "Reference" "#PWR054"
+		(property "Reference" "#PWR057"
 			(at 162.56 156.21 0)
 			(effects
@@
 			(project "LiF_FC-PCB_rev1"
 				(path "/9e3e8da7-e506-46c9-90e5-307e4ad30d29/17577359-df8d-4d28-9071-787d31b1b6da"
-					(reference "#PWR054")
+					(reference "#PWR057")
 					(unit 1)
 				)
@@
 		(on_board yes)
 		(dnp no)
-		(property "Reference" "#PWR049"
+		(property "Reference" "#PWR052"
 			(at 53.34 152.4 0)
 			(effects
@@
 			(project "LiF_FC-PCB_rev1"
 				(path "/9e3e8da7-e506-46c9-90e5-307e4ad30d29/17577359-df8d-4d28-9071-787d31b1b6da"
-					(reference "#PWR049")
+					(reference "#PWR052")
 					(unit 1)
 				)
@@
 		(on_board yes)
 		(dnp no)
-		(property "Reference" "J15"
+		(property "Reference" "J18"
 			(at 55.372 72.644 90)
 			(effects
@@
 			(project "LiF_FC-PCB_rev1"
 				(path "/9e3e8da7-e506-46c9-90e5-307e4ad30d29/17577359-df8d-4d28-9071-787d31b1b6da"
-					(reference "J15")
+					(reference "J18")
 					(unit 1)
 				)
@@
 		(on_board yes)
 		(dnp no)
-		(property "Reference" "#PWR052"
+		(property "Reference" "#PWR055"
 			(at 130.81 156.21 0)
 			(effects
@@
 			(project "LiF_FC-PCB_rev1"
 				(path "/9e3e8da7-e506-46c9-90e5-307e4ad30d29/17577359-df8d-4d28-9071-787d31b1b6da"
-					(reference "#PWR052")
+					(reference "#PWR055")
 					(unit 1)
 				)
@@
 		(on_board yes)
 		(dnp no)
-		(property "Reference" "TP18"
+		(property "Reference" "TP21"
 			(at 156.972 121.158 0)
 			(effects
@@
 			(project "LiF_FC-PCB_rev1"
 				(path "/9e3e8da7-e506-46c9-90e5-307e4ad30d29/17577359-df8d-4d28-9071-787d31b1b6da"
-					(reference "TP18")
+					(reference "TP21")
 					(unit 1)
 				)
@@
 		(on_board yes)
 		(dnp no)
-		(property "Reference" "TP16"
+		(property "Reference" "TP19"
 			(at 137.668 87.122 0)
 			(effects
@@
 			(project "LiF_FC-PCB_rev1"
 				(path "/9e3e8da7-e506-46c9-90e5-307e4ad30d29/17577359-df8d-4d28-9071-787d31b1b6da"
-					(reference "TP16")
+					(reference "TP19")
 					(unit 1)
 				)
@@
 		(on_board yes)
 		(dnp no)
-		(property "Reference" "#PWR050"
+		(property "Reference" "#PWR053"
 			(at 59.69 152.4 0)
 			(effects
@@
 			(project "LiF_FC-PCB_rev1"
 				(path "/9e3e8da7-e506-46c9-90e5-307e4ad30d29/17577359-df8d-4d28-9071-787d31b1b6da"
-					(reference "#PWR050")
+					(reference "#PWR053")
 					(unit 1)
 				)
@@
 		(on_board yes)
 		(dnp no)
-		(property "Reference" "J14"
+		(property "Reference" "J17"
 			(at 55.372 56.134 90)
 			(effects
@@
 			(project "LiF_FC-PCB_rev1"
 				(path "/9e3e8da7-e506-46c9-90e5-307e4ad30d29/17577359-df8d-4d28-9071-787d31b1b6da"
-					(reference "J14")
+					(reference "J17")
 					(unit 1)
 				)
@@
 		(on_board yes)
 		(dnp no)
-		(property "Reference" "#PWR044"
+		(property "Reference" "#PWR047"
 			(at 147.32 63.5 0)
 			(effects
@@
 			(project "LiF_FC-PCB_rev1"
 				(path "/9e3e8da7-e506-46c9-90e5-307e4ad30d29/17577359-df8d-4d28-9071-787d31b1b6da"
-					(reference "#PWR044")
+					(reference "#PWR047")
 					(unit 1)
 				)
@@
 		(on_board yes)
 		(dnp no)
-		(property "Reference" "#PWR055"
+		(property "Reference" "#PWR058"
 			(at 168.91 156.21 0)
 			(effects
@@
 			(project "LiF_FC-PCB_rev1"
 				(path "/9e3e8da7-e506-46c9-90e5-307e4ad30d29/17577359-df8d-4d28-9071-787d31b1b6da"
-					(reference "#PWR055")
+					(reference "#PWR058")
 					(unit 1)
 				)
@@
 		(on_board yes)
 		(dnp no)
-		(property "Reference" "#PWR047"
+		(property "Reference" "#PWR050"
 			(at 153.67 95.25 0)
 			(effects
@@
 			(project "LiF_FC-PCB_rev1"
 				(path "/9e3e8da7-e506-46c9-90e5-307e4ad30d29/17577359-df8d-4d28-9071-787d31b1b6da"
-					(reference "#PWR047")
+					(reference "#PWR050")
 					(unit 1)
 				)
@@
 		(on_board yes)
 		(dnp no)
-		(property "Reference" "#PWR053"
+		(property "Reference" "#PWR056"
 			(at 149.86 156.21 0)
 			(effects
@@
 			(project "LiF_FC-PCB_rev1"
 				(path "/9e3e8da7-e506-46c9-90e5-307e4ad30d29/17577359-df8d-4d28-9071-787d31b1b6da"
-					(reference "#PWR053")
+					(reference "#PWR056")
 					(unit 1)
 				)
@@
 		(on_board yes)
 		(dnp no)
-		(property "Reference" "J16"
+		(property "Reference" "J19"
 			(at 22.86 121.92 0)
 			(effects
@@
 			(project ""
 				(path "/9e3e8da7-e506-46c9-90e5-307e4ad30d29/17577359-df8d-4d28-9071-787d31b1b6da"
-					(reference "J16")
+					(reference "J19")
 					(unit 1)
 				)
@@
 		(on_board yes)
 		(dnp no)
-		(property "Reference" "#PWR051"
+		(property "Reference" "#PWR054"
 			(at 109.22 156.21 0)
 			(effects
@@
 			(project "LiF_FC-PCB_rev1"
 				(path "/9e3e8da7-e506-46c9-90e5-307e4ad30d29/17577359-df8d-4d28-9071-787d31b1b6da"
-					(reference "#PWR051")
-					(unit 1)
-				)
+					(reference "#PWR054")
+					(unit 1)
+				)

Commit message: set up board configuration and started routing PCB
Parts:
- TP15, TP16, TP17, TP18, TP19, TP20, TP21: footprint TestPoint:TestPoint_Bridge_Pitch2.54mm_Drill1.0mm -> TestPoint:TestPoint_Loop_D1.80mm_Drill1.0mm_Beaded
Changed lines of the file:
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@@
 			)
 		)
-		(property "Footprint" "TestPoint:TestPoint_Bridge_Pitch2.54mm_Drill1.0mm"
+		(property "Footprint" "TestPoint:TestPoint_Loop_D1.80mm_Drill1.0mm_Beaded"
 			(at 140.97 62.23 0)
 			(effects
@@
 			)
 		)
-		(property "Footprint" "TestPoint:TestPoint_Bridge_Pitch2.54mm_Drill1.0mm"
+		(property "Footprint" "TestPoint:TestPoint_Loop_D1.80mm_Drill1.0mm_Beaded"
 			(at 209.55 62.23 0)
 			(effects
@@
 			)
 		)
-		(property "Footprint" "TestPoint:TestPoint_Bridge_Pitch2.54mm_Drill1.0mm"
+		(property "Footprint" "TestPoint:TestPoint_Loop_D1.80mm_Drill1.0mm_Beaded"
 			(at 274.32 64.77 0)
 			(effects
@@
 			)
 		)
-		(property "Footprint" "TestPoint:TestPoint_Bridge_Pitch2.54mm_Drill1.0mm"
+		(property "Footprint" "TestPoint:TestPoint_Loop_D1.80mm_Drill1.0mm_Beaded"
 			(at 181.61 119.38 0)
 			(effects
@@
 			)
 		)
-		(property "Footprint" "TestPoint:TestPoint_Bridge_Pitch2.54mm_Drill1.0mm"
+		(property "Footprint" "TestPoint:TestPoint_Loop_D1.80mm_Drill1.0mm_Beaded"
 			(at 194.31 64.77 0)
 			(effects
@@
 			)
 		)
-		(property "Footprint" "TestPoint:TestPoint_Bridge_Pitch2.54mm_Drill1.0mm"
+		(property "Footprint" "TestPoint:TestPoint_Loop_D1.80mm_Drill1.0mm_Beaded"
 			(at 153.67 125.73 0)
 			(effects
@@
 			)
 		)
-		(property "Footprint" "TestPoint:TestPoint_Bridge_Pitch2.54mm_Drill1.0mm"
+		(property "Footprint" "TestPoint:TestPoint_Loop_D1.80mm_Drill1.0mm_Beaded"
 			(at 140.97 82.55 0)
 			(effects

Commit message: backup before expanding the board size
Parts:
- TP16, TP20: value GND -> GNDA
- TP18: value FLT -> LC_FLT
Changed lines of the file:
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@@
 			)
 		)
-		(property "Value" "GND"
+		(property "Value" "GNDA"
 			(at 206.248 60.198 0)
 			(effects
@@
 			)
 		)
-		(property "Value" "FLT"
+		(property "Value" "LC_FLT"
 			(at 271.018 62.738 0)
 			(effects
@@
 			)
 		)
-		(property "Value" "GND"
+		(property "Value" "GNDA"
 			(at 178.308 117.348 0)
 			(effects

Commit message: backup before leaving school
Parts:
- J17, J18: footprint Connector_PinHeader_2.54mm:PinHeader_1x02_P2.54mm_Vertical -> Connector_PinHeader_2.54mm:PinHeader_1x02_P2.54mm_Vertical_SMD_Pin1Left
Changed lines of the file:
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@@
 			)
 		)
-		(property "Footprint" "Connector_PinHeader_2.54mm:PinHeader_1x02_P2.54mm_Vertical"
+		(property "Footprint" "Connector_PinHeader_2.54mm:PinHeader_1x02_P2.54mm_Vertical_SMD_Pin1Left"
 			(at 54.61 73.66 0)
 			(effects
@@
 			)
 		)
-		(property "Footprint" "Connector_PinHeader_2.54mm:PinHeader_1x02_P2.54mm_Vertical"
+		(property "Footprint" "Connector_PinHeader_2.54mm:PinHeader_1x02_P2.54mm_Vertical_SMD_Pin1Left"
 			(at 54.61 57.15 0)
 			(effects
