File: KiCAD/LiF_FC-PCB_rev1/LiF_PowerReg.kicad_sch (KiCad schematic)
At the start: 45 parts, among them J1 VCAN_{EN}, J10 R3V3_{EN}, J11 A3V3_{EN}, J2 R5V0_{EN}, J3 REG V_{IN} EN, J4 Barrel Jack, J5 CAN USB_{EN}, J6 PROG USB_{EN}, J7 V_{IN}, J8 3V3 REG_{EN}, J9 A3V3 REG_{EN}, U1 AZ1117-3.3, U2 AZ1117-3.3

Commit message: progress backup before increasing the size of the PCB again
Parts:
- J2, J5: footprint Connector_PinHeader_2.54mm:PinHeader_1x02_P2.54mm_Vertical_SMD_Pin1Left -> Connector_PinHeader_2.54mm:PinHeader_1x02_P2.54mm_Vertical
- J3: now not fitted; now left out of the parts list
- R3: now left out of the parts list
Connections:
- net 5V Regulator/V_{IN}: now also D1.1 (K), D2.1 (K), J3.2 (Pin_2), R3.2
- net GND: now also J7.1 (Pin_1); no longer J7.2 (Pin_2)
- net V_{supply}: now also J7.2 (Pin_2); no longer J7.1 (Pin_1)
Other:
- moved on the sheet: J7
Changed lines of the file:
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@@
 	)
 	(junction
+		(at 57.15 69.85)
+		(diameter 0)
+		(color 0 0 0 0)
+	)
+	(junction
 		(at 123.19 59.69)
 		(diameter 0)
@@
 	)
 	(junction
+		(at 69.85 69.85)
+		(diameter 0)
+		(color 0 0 0 0)
+	)
+	(junction
 		(at 176.53 128.27)
 		(diameter 0)
@@
 	(wire
 		(pts
+			(xy 69.85 69.85) (xy 77.47 69.85)
+		)
+		(stroke
+			(width 0)
+			(type default)
+		)
+	)
+	(wire
+		(pts
 			(xy 191.77 144.78) (xy 191.77 148.59)
 		)
@@
 	(wire
 		(pts
+			(xy 57.15 69.85) (xy 57.15 77.47)
+		)
+		(stroke
+			(width 0)
+			(type default)
+		)
+	)
+	(wire
+		(pts
 			(xy 256.54 134.62) (xy 259.08 134.62)
 		)
@@
 	(wire
 		(pts
+			(xy 69.85 77.47) (xy 69.85 69.85)
+		)
+		(stroke
+			(width 0)
+			(type default)
+		)
+	)
+	(wire
+		(pts
 			(xy 123.19 59.69) (xy 127 59.69)
 		)
@@
 	(wire
 		(pts
+			(xy 57.15 77.47) (xy 69.85 77.47)
+		)
+		(stroke
+			(width 0)
+			(type default)
+		)
+	)
+	(wire
+		(pts
 			(xy 246.38 71.12) (xy 248.92 71.12)
 		)
@@
 	(wire
 		(pts
+			(xy 57.15 69.85) (xy 58.42 69.85)
+		)
+		(stroke
+			(width 0)
+			(type default)
+		)
+	)
+	(wire
+		(pts
 			(xy 77.47 69.85) (xy 78.74 69.85)
 		)
@@
 	(wire
 		(pts
-			(xy 50.8 69.85) (xy 58.42 69.85)
+			(xy 50.8 69.85) (xy 57.15 69.85)
 		)
 		(stroke
@@
 	(wire
 		(pts
-			(xy 68.58 69.85) (xy 77.47 69.85)
+			(xy 68.58 69.85) (xy 69.85 69.85)
 		)
 		(stroke
@@
 			)
 		)
-		(property "Footprint" "Connector_PinHeader_2.54mm:PinHeader_1x02_P2.54mm_Vertical_SMD_Pin1Left"
+		(property "Footprint" "Connector_PinHeader_2.54mm:PinHeader_1x02_P2.54mm_Vertical"
 			(at 129.54 52.07 0)
 			(effects
@@
 		(unit 1)
 		(exclude_from_sim no)
-		(in_bom yes)
-		(on_board yes)
+		(in_bom no)
+		(on_board no)
 		(dnp yes)
 		(property "Reference" "R3"
@@
 		(unit 1)
 		(exclude_from_sim no)
-		(in_bom yes)
-		(on_board yes)
-		(dnp no)
+		(in_bom no)
+		(on_board no)
+		(dnp yes)
 		(property "Reference" "J3"
 			(at 65.532 59.944 90)
@@
 			)
 		)
-		(property "Footprint" "Connector_PinHeader_2.54mm:PinHeader_1x02_P2.54mm_Vertical_SMD_Pin1Left"
+		(property "Footprint" "Connector_PinHeader_2.54mm:PinHeader_1x02_P2.54mm_Vertical"
 			(at 129.54 72.39 0)
 			(effects
@@
 	(symbol
 		(lib_id "Connector_Generic:Conn_01x02")
-		(at 24.13 82.55 0)
-		(mirror y)
+		(at 24.13 85.09 180)
 		(unit 1)
 		(exclude_from_sim no)
@@
 		(dnp no)
 		(property "Reference" "J7"
-			(at 24.13 88.646 0)
+			(at 24.13 78.994 0)
 			(effects
 				(font
@@
 		)
 		(property "Value" "V_{IN}"
-			(at 24.13 91.186 0)
+			(at 24.13 76.454 0)
 			(effects
 				(font
@@
 		)
 		(property "Footprint" "Connector_JST:JST_PH_B2B-PH-K_1x02_P2.00mm_Vertical"
-			(at 24.13 82.55 0)
+			(at 24.13 85.09 0)
 			(effects
 				(font
@@
 		)
 		(property "Datasheet" "~"
-			(at 24.13 82.55 0)
+			(at 24.13 85.09 0)
 			(effects
 				(font
@@
 		)
 		(property "Description" "Generic connector, single row, 01x02, script generated (kicad-library-utils/schlib/autogen/connector/)"
-			(at 24.13 82.55 0)
+			(at 24.13 85.09 0)
 			(effects
 				(font
@@
 		)
 		(instances
-			(project ""
+			(project "LiF_FC-PCB_rev1"
 				(path "/9e3e8da7-e506-46c9-90e5-307e4ad30d29/dbf56dc2-3990-4801-b0e0-f59d351af64c"
 					(reference "J7")

Commit message: Created new KiCAD project for IO PCB, moved relevant components there, saving backup before reannotating the Service PCB schematics
Parts:
- J1, J10, J11, J2, J5, J6, J8, J9: now not fitted; now left out of the parts list

Commit message: finished service PCB routing and silkscreen, finished IO PCB layout, routing, and silkscreen. Exported production files, submitted PCB for manufacturing by JLCPCB
Parts:
- removed TP3, TP8: GND, TestPoint:TestPoint_Loop_D1.80mm_Drill1.0mm_Beaded, symbol Connector:TestPoint
