File: KiCAD/LiF_FC-PCB_rev1/LiF_7Seg.kicad_sch (KiCad schematic)
At the start: 7 parts, among them J37 BTN 3V3_{EN}, U13 DC56-11EWA, U14 NCA9555

Commit message: Created new KiCAD project for IO PCB, moved relevant components there, saving backup before reannotating the Service PCB schematics
Parts:
- removed RN1, RN2: 8x 470, LiF_PCB_Footprints:RESCAXE50P380X160X55-16N, symbol LiF_PCB_Symbols:EXB-2HV471JV
- removed U13: DC56-11EWA, Display_7Segment:DA56-11SURKWA, symbol Display_Character:DC56-11EWA
- J37: now not fitted; now left out of the parts list
Connections:
- net DIG1_A renamed IO0
- net DIG1_B renamed IO1
- net DIG1_C renamed IO2
- net DIG1_D renamed IO3
- net DIG1_DP renamed IO7
- net DIG1_E renamed IO4
- net DIG1_F renamed IO5
- net DIG1_G renamed IO6
- net DIG2_A renamed IO8
- net DIG2_B renamed IO9
- net DIG2_C renamed IO10
- net DIG2_D renamed IO11
- net DIG2_DP renamed IO15
- net DIG2_E renamed IO12
- net DIG2_F renamed IO13
- net DIG2_G renamed IO14
Other:
- note added: "DIG1_A"
- note added: "DIG1_B"
- note added: "DIG1_C"
- note added: "DIG1_D"
- note added: "DIG1_DP"
- note added: "DIG1_E"
- note added: "DIG1_F"
- note added: "DIG1_G"
- note added: "DIG2_A"
- note added: "DIG2_B"
- note added: "DIG2_C"
- note added: "DIG2_D"
- note added: "DIG2_DP"
- note added: "DIG2_E"
- note added: "DIG2_F"
- note added: "DIG2_G"
- note removed: "7-Segment Display"

Commit message: backup before redoing the analog section
Parts:
- renumbered C42 to C43, J37 to J38, U14 to U13
Changed lines of the file:
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@@
 		(on_board no)
 		(dnp yes)
-		(property "Reference" "J37"
+		(property "Reference" "J38"
 			(at 47.752 49.784 90)
 			(effects
@@
 			(project "LiF_FC-PCB_rev1"
 				(path "/9e3e8da7-e506-46c9-90e5-307e4ad30d29/d823ad92-d1a3-4f4d-8dfc-d728d5836dc0"
-					(reference "J37")
+					(reference "J38")
 					(unit 1)
 				)
@@
 		(dnp no)
 		(fields_autoplaced yes)
-		(property "Reference" "#PWR086"
+		(property "Reference" "#PWR085"
 			(at 120.65 140.97 0)
 			(effects
@@
 			(project "LiF_FC-PCB_rev1"
 				(path "/9e3e8da7-e506-46c9-90e5-307e4ad30d29/d823ad92-d1a3-4f4d-8dfc-d728d5836dc0"
-					(reference "#PWR086")
+					(reference "#PWR085")
 					(unit 1)
 				)
@@
 		(on_board yes)
 		(dnp no)
-		(property "Reference" "U14"
+		(property "Reference" "U13"
 			(at 112.522 80.772 0)
 			(effects
@@
 			(project "LiF_FC-PCB_rev1"
 				(path "/9e3e8da7-e506-46c9-90e5-307e4ad30d29/d823ad92-d1a3-4f4d-8dfc-d728d5836dc0"
-					(reference "U14")
+					(reference "U13")
 					(unit 1)
 				)
@@
 		(on_board yes)
 		(dnp no)
-		(property "Reference" "C42"
+		(property "Reference" "C43"
 			(at 111.76 66.0399 0)
 			(effects
@@
 			(project "LiF_FC-PCB_rev1"
 				(path "/9e3e8da7-e506-46c9-90e5-307e4ad30d29/d823ad92-d1a3-4f4d-8dfc-d728d5836dc0"
-					(reference "C42")
+					(reference "C43")
 					(unit 1)
 				)
@@
 		(on_board yes)
 		(dnp no)
-		(property "Reference" "#PWR085"
+		(property "Reference" "#PWR084"
 			(at 106.68 140.97 0)
 			(effects
@@
 			(project "LiF_FC-PCB_rev1"
 				(path "/9e3e8da7-e506-46c9-90e5-307e4ad30d29/d823ad92-d1a3-4f4d-8dfc-d728d5836dc0"
-					(reference "#PWR085")
+					(reference "#PWR084")
 					(unit 1)
 				)
@@
 		(dnp no)
 		(fields_autoplaced yes)
-		(property "Reference" "#PWR082"
+		(property "Reference" "#PWR083"
 			(at 115.57 78.74 0)
 			(effects
@@
 			(project "LiF_FC-PCB_rev1"
 				(path "/9e3e8da7-e506-46c9-90e5-307e4ad30d29/d823ad92-d1a3-4f4d-8dfc-d728d5836dc0"
-					(reference "#PWR082")
+					(reference "#PWR083")
 					(unit 1)
 				)
