File: KiCAD/LiF_FC-PCB_rev1/LiF_ACC.kicad_sch (KiCad schematic)
At the start: 0 parts

Commit message: Finished schematics, mostly. Only MCU sheet left. Doing component sourcing
Parts:
- added C07_1, C07_2: 0.1u, Capacitor_SMD:C_0805_2012Metric, symbol Device:C
- added J27: ACC 3V3_{EN}, Connector_PinHeader_2.54mm:PinHeader_1x02_P2.54mm_Vertical, symbol Connector:Conn_01x02_Pin
- added R53: 0, Resistor_SMD:R_0805_2012Metric, symbol Device:R
- added U11: BMA400, LiF_PCB_Footprints:XDCR_BMA400, symbol LiF_PCB_Symbols:BMA400
Connections:
- new net 3V3_{IN}: J27.2 (Pin_2), R53.2
- new net ACC_3V3: C07_1.1, C07_2.1, J27.1 (Pin_1), R53.1, U11.10 (~{CSB}), U11.3 (VDDIO), U11.7 (VDD)
- new net ACC_INT1: U11.5 (INT1)
- new net ACC_INT2: U11.6 (INT2)
- new net GND: C07_1.2, C07_2.2, U11.1 (SDO), U11.8 (GNDIO), U11.9 (GND)
- new net I2C.SCL: U11.12 (SCX)
- new net I2C.SDA: U11.2 (SDX)
Other:
- note added: "Accelerometer IC"
- note added: "CSB to high puts the IC into I2C mode as the default is SPI"
- note added: "Datasheet recommends adding cap to GND for both"
- note added: "ESP32_GPIO"
- note added: "ESP32_SCL Pin"
- note added: "ESP32_SDA Pin"
- note added: "I2C 4.7k Pull-Ups moved to MCU sheet"
- note added: "Inputs"
- note added: "Interrupt Flags"
- note added: "Lithium Firefly - Accelerometer"
- note added: "Only one INT pin is required We can connect both anyway INT1 = free-fall condition INT2 = excessive accel or sudden stop (like a crash)"
- note added: "Power Input"
- note added: "SDO to GND sets it to address bit 0 This gives 7-bit I2C address of 0x14"
- note added: "VDD = IC power VDDIO = IO (I2C) power Both are using 3V3 here"
- company: (none) -> Lithium Firefly Team
- title: (none) -> LiF - Accelerometer

Commit message: Added MCU pinout, shanged shift registers to GPIO expanders to save pins on MCU
Parts:
- renumbered J27 to J28, R53 to R54
Other:
- title: LiF - Accelerometer -> Lithium Firefly Custom FC/CC PCB

Commit message: Finalized schematic diagram. Only needs formatting fixes and resistor component sourcing info
Parts:
- renumbered C07_1 to C35, C07_2 to C36, J28 to J31
Changed lines of the file:
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@@
 		(dnp no)
 		(fields_autoplaced yes)
-		(property "Reference" "#PWR068"
+		(property "Reference" "#PWR071"
 			(at 158.75 90.17 0)
 			(effects
@@
 			(project "LiF_FC-PCB_rev1"
 				(path "/9e3e8da7-e506-46c9-90e5-307e4ad30d29/25eacf96-1a70-4276-a4a6-d0196807ae93"
-					(reference "#PWR068")
+					(reference "#PWR071")
 					(unit 1)
 				)
@@
 		(dnp no)
 		(fields_autoplaced yes)
-		(property "Reference" "#PWR069"
+		(property "Reference" "#PWR072"
 			(at 175.26 90.17 0)
 			(effects
@@
 			(project "LiF_FC-PCB_rev1"
 				(path "/9e3e8da7-e506-46c9-90e5-307e4ad30d29/25eacf96-1a70-4276-a4a6-d0196807ae93"
-					(reference "#PWR069")
+					(reference "#PWR072")
 					(unit 1)
 				)
@@
 		(on_board yes)
 		(dnp no)
-		(property "Reference" "J28"
+		(property "Reference" "J31"
 			(at 62.992 66.294 90)
 			(effects
@@
 			(project "LiF_FC-PCB_rev1"
 				(path "/9e3e8da7-e506-46c9-90e5-307e4ad30d29/25eacf96-1a70-4276-a4a6-d0196807ae93"
-					(reference "J28")
+					(reference "J31")
 					(unit 1)
 				)
@@
 		(on_board yes)
 		(dnp no)
-		(property "Reference" "C07_2"
+		(property "Reference" "C36"
 			(at 184.912 77.978 0)
 			(effects
@@
 			(project "LiF_FC-PCB_rev1"
 				(path "/9e3e8da7-e506-46c9-90e5-307e4ad30d29/25eacf96-1a70-4276-a4a6-d0196807ae93"
-					(reference "C07_2")
+					(reference "C36")
 					(unit 1)
 				)
@@
 		(dnp no)
 		(fields_autoplaced yes)
-		(property "Reference" "#PWR071"
+		(property "Reference" "#PWR074"
 			(at 167.64 146.05 0)
 			(effects
@@
 			(project "LiF_FC-PCB_rev1"
 				(path "/9e3e8da7-e506-46c9-90e5-307e4ad30d29/25eacf96-1a70-4276-a4a6-d0196807ae93"
-					(reference "#PWR071")
+					(reference "#PWR074")
 					(unit 1)
 				)
@@
 		(on_board yes)
 		(dnp no)
-		(property "Reference" "C07_1"
+		(property "Reference" "C35"
 			(at 154.94 77.724 0)
 			(effects
@@
 			(project "LiF_FC-PCB_rev1"
 				(path "/9e3e8da7-e506-46c9-90e5-307e4ad30d29/25eacf96-1a70-4276-a4a6-d0196807ae93"
-					(reference "C07_1")
+					(reference "C35")
 					(unit 1)
 				)
@@
 		(dnp no)
 		(fields_autoplaced yes)
-		(property "Reference" "#PWR070"
+		(property "Reference" "#PWR073"
 			(at 151.13 134.62 0)
 			(effects
@@
 			(project "LiF_FC-PCB_rev1"
 				(path "/9e3e8da7-e506-46c9-90e5-307e4ad30d29/25eacf96-1a70-4276-a4a6-d0196807ae93"
-					(reference "#PWR070")
-					(unit 1)
-				)
+					(reference "#PWR073")
+					(unit 1)
+				)

Commit message: backup before leaving school
Parts:
- J31: footprint Connector_PinHeader_2.54mm:PinHeader_1x02_P2.54mm_Vertical -> Connector_PinHeader_2.54mm:PinHeader_1x02_P2.54mm_Vertical_SMD_Pin1Left
Changed lines of the file:
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@@
 			)
 		)
-		(property "Footprint" "Connector_PinHeader_2.54mm:PinHeader_1x02_P2.54mm_Vertical"
+		(property "Footprint" "Connector_PinHeader_2.54mm:PinHeader_1x02_P2.54mm_Vertical_SMD_Pin1Left"
 			(at 62.23 67.31 0)
 			(effects

Commit message: Created new KiCAD project for IO PCB, moved relevant components there, saving backup before reannotating the Service PCB schematics
Parts:
- J31: now not fitted; now left out of the parts list

Commit message: backup before redoing the analog section
Parts:
- renumbered J31 to J32
Changed lines of the file:
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@@
 		(dnp no)
 		(fields_autoplaced yes)
-		(property "Reference" "#PWR071"
+		(property "Reference" "#PWR072"
 			(at 158.75 90.17 0)
 			(effects
@@
 			(project "LiF_FC-PCB_rev1"
 				(path "/9e3e8da7-e506-46c9-90e5-307e4ad30d29/25eacf96-1a70-4276-a4a6-d0196807ae93"
-					(reference "#PWR071")
+					(reference "#PWR072")
 					(unit 1)
 				)
@@
 		(dnp no)
 		(fields_autoplaced yes)
-		(property "Reference" "#PWR072"
+		(property "Reference" "#PWR073"
 			(at 175.26 90.17 0)
 			(effects
@@
 			(project "LiF_FC-PCB_rev1"
 				(path "/9e3e8da7-e506-46c9-90e5-307e4ad30d29/25eacf96-1a70-4276-a4a6-d0196807ae93"
-					(reference "#PWR072")
+					(reference "#PWR073")
 					(unit 1)
 				)
@@
 		(on_board no)
 		(dnp yes)
-		(property "Reference" "J31"
+		(property "Reference" "J32"
 			(at 62.992 66.294 90)
 			(effects
@@
 			(project "LiF_FC-PCB_rev1"
 				(path "/9e3e8da7-e506-46c9-90e5-307e4ad30d29/25eacf96-1a70-4276-a4a6-d0196807ae93"
-					(reference "J31")
+					(reference "J32")
 					(unit 1)
 				)
@@
 		(dnp no)
 		(fields_autoplaced yes)
-		(property "Reference" "#PWR074"
+		(property "Reference" "#PWR075"
 			(at 167.64 146.05 0)
 			(effects
@@
 			(project "LiF_FC-PCB_rev1"
 				(path "/9e3e8da7-e506-46c9-90e5-307e4ad30d29/25eacf96-1a70-4276-a4a6-d0196807ae93"
-					(reference "#PWR074")
+					(reference "#PWR075")
 					(unit 1)
 				)
@@
 		(dnp no)
 		(fields_autoplaced yes)
-		(property "Reference" "#PWR073"
+		(property "Reference" "#PWR074"
 			(at 151.13 134.62 0)
 			(effects
@@
 			(project "LiF_FC-PCB_rev1"
 				(path "/9e3e8da7-e506-46c9-90e5-307e4ad30d29/25eacf96-1a70-4276-a4a6-d0196807ae93"
-					(reference "#PWR073")
+					(reference "#PWR074")
 					(unit 1)
 				)
