File: KiCAD/LiF_FC-PCB_rev1/LiF_Audio.kicad_sch (KiCad schematic)
At the start: 24 parts, among them J32 Amp V select, J33 ST 1 Bypass, J34 ST 2 Bypass, J35 Vol Pot Bypass, J36 SKP OUT, U12 PAM8302AAS

Commit message: backup before redoing the analog section
Parts:
- renumbered C58 to C40, C40 to C41, C41 to C42, J32 to J33, J33 to J34, J34 to J35, J35 to J36, J36 to J37
Changed lines of the file:
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@@
 		(dnp no)
 		(fields_autoplaced yes)
-		(property "Reference" "#PWR081"
+		(property "Reference" "#PWR082"
 			(at 228.6 158.75 0)
 			(effects
@@
 			(project "LiF_FC-PCB_rev1"
 				(path "/9e3e8da7-e506-46c9-90e5-307e4ad30d29/75541181-887f-448c-8628-82c2df7284ca"
-					(reference "#PWR081")
+					(reference "#PWR082")
 					(unit 1)
 				)
@@
 		(on_board yes)
 		(dnp no)
-		(property "Reference" "C40"
+		(property "Reference" "C41"
 			(at 67.31 138.4299 0)
 			(effects
@@
 			(project "LiF_FC-PCB_rev1"
 				(path "/9e3e8da7-e506-46c9-90e5-307e4ad30d29/75541181-887f-448c-8628-82c2df7284ca"
-					(reference "C40")
+					(reference "C41")
 					(unit 1)
 				)
@@
 		(on_board no)
 		(dnp yes)
-		(property "Reference" "J34"
+		(property "Reference" "J35"
 			(at 78.994 105.664 90)
 			(effects
@@
 			(project "LiF_FC-PCB_rev1"
 				(path "/9e3e8da7-e506-46c9-90e5-307e4ad30d29/75541181-887f-448c-8628-82c2df7284ca"
-					(reference "J34")
+					(reference "J35")
 					(unit 1)
 				)
@@
 		(dnp no)
 		(fields_autoplaced yes)
-		(property "Reference" "#PWR078"
+		(property "Reference" "#PWR079"
 			(at 87.63 152.4 0)
 			(effects
@@
 			(project "LiF_FC-PCB_rev1"
 				(path "/9e3e8da7-e506-46c9-90e5-307e4ad30d29/75541181-887f-448c-8628-82c2df7284ca"
-					(reference "#PWR078")
+					(reference "#PWR079")
 					(unit 1)
 				)
@@
 		(on_board no)
 		(dnp yes)
-		(property "Reference" "J33"
+		(property "Reference" "J34"
 			(at 62.484 105.664 90)
 			(effects
@@
 			(project "LiF_FC-PCB_rev1"
 				(path "/9e3e8da7-e506-46c9-90e5-307e4ad30d29/75541181-887f-448c-8628-82c2df7284ca"
-					(reference "J33")
+					(reference "J34")
 					(unit 1)
 				)
@@
 		(dnp yes)
 		(fields_autoplaced yes)
-		(property "Reference" "J32"
+		(property "Reference" "J33"
 			(at 58.42 40.64 90)
 			(effects
@@
 			(project "LiF_FC-PCB_rev1"
 				(path "/9e3e8da7-e506-46c9-90e5-307e4ad30d29/75541181-887f-448c-8628-82c2df7284ca"
-					(reference "J32")
+					(reference "J33")
 					(unit 1)
 				)
@@
 		(dnp no)
 		(fields_autoplaced yes)
-		(property "Reference" "J36"
+		(property "Reference" "J37"
 			(at 262.89 133.3499 0)
 			(effects
@@
 			(project "LiF_FC-PCB_rev1"
 				(path "/9e3e8da7-e506-46c9-90e5-307e4ad30d29/75541181-887f-448c-8628-82c2df7284ca"
-					(reference "J36")
+					(reference "J37")
 					(unit 1)
 				)
@@
 		(on_board yes)
 		(dnp no)
-		(property "Reference" "C58"
+		(property "Reference" "C40"
 			(at 166.37 141.732 90)
 			(effects
@@
 			(project "LiF_FC-PCB_rev1"
 				(path "/9e3e8da7-e506-46c9-90e5-307e4ad30d29/75541181-887f-448c-8628-82c2df7284ca"
-					(reference "C58")
+					(reference "C40")
 					(unit 1)
 				)
@@
 		(dnp no)
 		(fields_autoplaced yes)
-		(property "Reference" "#PWR079"
+		(property "Reference" "#PWR080"
 			(at 127 153.67 0)
 			(effects
@@
 			(project "LiF_FC-PCB_rev1"
 				(path "/9e3e8da7-e506-46c9-90e5-307e4ad30d29/75541181-887f-448c-8628-82c2df7284ca"
-					(reference "#PWR079")
+					(reference "#PWR080")
 					(unit 1)
 				)
@@
 		(dnp no)
 		(fields_autoplaced yes)
-		(property "Reference" "#PWR075"
+		(property "Reference" "#PWR076"
 			(at 213.36 121.92 0)
 			(effects
@@
 			(project "LiF_FC-PCB_rev1"
 				(path "/9e3e8da7-e506-46c9-90e5-307e4ad30d29/75541181-887f-448c-8628-82c2df7284ca"
-					(reference "#PWR075")
+					(reference "#PWR076")
 					(unit 1)
 				)
@@
 		(dnp no)
 		(fields_autoplaced yes)
-		(property "Reference" "#PWR077"
+		(property "Reference" "#PWR078"
 			(at 71.12 152.4 0)
 			(effects
@@
 			(project "LiF_FC-PCB_rev1"
 				(path "/9e3e8da7-e506-46c9-90e5-307e4ad30d29/75541181-887f-448c-8628-82c2df7284ca"
-					(reference "#PWR077")
+					(reference "#PWR078")
 					(unit 1)
 				)
@@
 		(dnp no)
 		(fields_autoplaced yes)
-		(property "Reference" "#PWR080"
+		(property "Reference" "#PWR081"
 			(at 205.74 158.75 0)
 			(effects
@@
 			(project "LiF_FC-PCB_rev1"
 				(path "/9e3e8da7-e506-46c9-90e5-307e4ad30d29/75541181-887f-448c-8628-82c2df7284ca"
-					(reference "#PWR080")
+					(reference "#PWR081")
 					(unit 1)
 				)
@@
 		(dnp no)
 		(fields_autoplaced yes)
-		(property "Reference" "#PWR076"
+		(property "Reference" "#PWR077"
 			(at 158.75 149.86 0)
 			(effects
@@
 			(project "LiF_FC-PCB_rev1"
 				(path "/9e3e8da7-e506-46c9-90e5-307e4ad30d29/75541181-887f-448c-8628-82c2df7284ca"
-					(reference "#PWR076")
+					(reference "#PWR077")
 					(unit 1)
 				)
@@
 		(on_board yes)
 		(dnp no)
-		(property "Reference" "C41"
+		(property "Reference" "C42"
 			(at 83.82 138.4299 0)
 			(effects
@@
 			(project "LiF_FC-PCB_rev1"
 				(path "/9e3e8da7-e506-46c9-90e5-307e4ad30d29/75541181-887f-448c-8628-82c2df7284ca"
-					(reference "C41")
+					(reference "C42")
 					(unit 1)
 				)
@@
 		(on_board no)
 		(dnp yes)
-		(property "Reference" "J35"
+		(property "Reference" "J36"
 			(at 123.444 105.664 90)
 			(effects
@@
 			(project "LiF_FC-PCB_rev1"
 				(path "/9e3e8da7-e506-46c9-90e5-307e4ad30d29/75541181-887f-448c-8628-82c2df7284ca"
-					(reference "J35")
+					(reference "J36")
 					(unit 1)
 				)
