File: KiCAD/LiF_FC-PCB_rev1/LiF_Buttons.kicad_sch (KiCad schematic)
At the start: 13 parts, among them J38 BTN 3V3_{EN}, J43 Door Closed, U15 SN74HC14DR, U16 SN74HC14DR, U17 NCA9555

Commit message: backup before redoing the analog section
Parts:
- renumbered C48 to C44, C49 to C45, C57 to C46, C53 to C47, J38 to J39, J43 to J40, R66 to R61, R76 to R62, R70 to R63, R77 to R64, U15 to U14, U16 to U15, U17 to U16
Changed lines of the file:
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@@
 		(dnp no)
 		(fields_autoplaced yes)
-		(property "Reference" "U15"
+		(property "Reference" "U14"
 			(at 105.41 34.29 0)
 			(effects
@@
 			(project "LiF_FC-PCB_rev1"
 				(path "/9e3e8da7-e506-46c9-90e5-307e4ad30d29/5a2c7040-8854-4895-b7b6-208daa06b69a"
-					(reference "U15")
+					(reference "U14")
 					(unit 1)
 				)
@@
 		(on_board yes)
 		(dnp no)
-		(property "Reference" "#PWR0107"
+		(property "Reference" "#PWR091"
 			(at 41.91 194.31 0)
 			(effects
@@
 			(project "LiF_FC-PCB_rev1"
 				(path "/9e3e8da7-e506-46c9-90e5-307e4ad30d29/5a2c7040-8854-4895-b7b6-208daa06b69a"
-					(reference "#PWR0107")
+					(reference "#PWR091")
 					(unit 1)
 				)
@@
 		(dnp no)
 		(fields_autoplaced yes)
-		(property "Reference" "#PWR0108"
+		(property "Reference" "#PWR092"
 			(at 55.88 194.31 0)
 			(effects
@@
 			(project "LiF_FC-PCB_rev1"
 				(path "/9e3e8da7-e506-46c9-90e5-307e4ad30d29/5a2c7040-8854-4895-b7b6-208daa06b69a"
-					(reference "#PWR0108")
+					(reference "#PWR092")
 					(unit 1)
 				)
@@
 		(dnp no)
 		(fields_autoplaced yes)
-		(property "Reference" "R77"
+		(property "Reference" "R64"
 			(at 213.36 139.7 90)
 			(effects
@@
 			(project "LiF_FC-PCB_rev1"
 				(path "/9e3e8da7-e506-46c9-90e5-307e4ad30d29/5a2c7040-8854-4895-b7b6-208daa06b69a"
-					(reference "R77")
+					(reference "R64")
 					(unit 1)
 				)
@@
 		(on_board yes)
 		(dnp no)
-		(property "Reference" "#PWR096"
+		(property "Reference" "#PWR086"
 			(at 219.71 119.38 0)
 			(effects
@@
 			(project "LiF_FC-PCB_rev1"
 				(path "/9e3e8da7-e506-46c9-90e5-307e4ad30d29/5a2c7040-8854-4895-b7b6-208daa06b69a"
-					(reference "#PWR096")
+					(reference "#PWR086")
 					(unit 1)
 				)
@@
 		(dnp no)
 		(fields_autoplaced yes)
-		(property "Reference" "U16"
+		(property "Reference" "U15"
 			(at 105.41 142.24 0)
 			(effects
@@
 			(project "LiF_FC-PCB_rev1"
 				(path "/9e3e8da7-e506-46c9-90e5-307e4ad30d29/5a2c7040-8854-4895-b7b6-208daa06b69a"
-					(reference "U16")
+					(reference "U15")
 					(unit 2)
 				)
@@
 		(on_board yes)
 		(dnp no)
-		(property "Reference" "U17"
+		(property "Reference" "U16"
 			(at 47.752 134.112 0)
 			(effects
@@
 			(project "LiF_FC-PCB_rev1"
 				(path "/9e3e8da7-e506-46c9-90e5-307e4ad30d29/5a2c7040-8854-4895-b7b6-208daa06b69a"
-					(reference "U17")
+					(reference "U16")
 					(unit 1)
 				)
@@
 		(on_board yes)
 		(dnp no)
-		(property "Reference" "C48"
+		(property "Reference" "C44"
 			(at 210.82 96.5199 0)
 			(effects
@@
 			(project "LiF_FC-PCB_rev1"
 				(path "/9e3e8da7-e506-46c9-90e5-307e4ad30d29/5a2c7040-8854-4895-b7b6-208daa06b69a"
-					(reference "C48")
+					(reference "C44")
 					(unit 1)
 				)
@@
 		(on_board yes)
 		(dnp no)
-		(property "Reference" "C57"
+		(property "Reference" "C46"
 			(at 224.028 151.13 0)
 			(effects
@@
 			(project "LiF_FC-PCB_rev1"
 				(path "/9e3e8da7-e506-46c9-90e5-307e4ad30d29/5a2c7040-8854-4895-b7b6-208daa06b69a"
-					(reference "C57")
+					(reference "C46")
 					(unit 1)
 				)
@@
 		(dnp no)
 		(fields_autoplaced yes)
-		(property "Reference" "U16"
+		(property "Reference" "U15"
 			(at 243.84 137.16 0)
 			(effects
@@
 			(project "LiF_FC-PCB_rev1"
 				(path "/9e3e8da7-e506-46c9-90e5-307e4ad30d29/5a2c7040-8854-4895-b7b6-208daa06b69a"
-					(reference "U16")
+					(reference "U15")
 					(unit 6)
 				)
@@
 		(on_board yes)
 		(dnp no)
-		(property "Reference" "U16"
+		(property "Reference" "U15"
 			(at 262.636 83.82 0)
 			(effects
@@
 			(project "LiF_FC-PCB_rev1"
 				(path "/9e3e8da7-e506-46c9-90e5-307e4ad30d29/5a2c7040-8854-4895-b7b6-208daa06b69a"
-					(reference "U16")
+					(reference "U15")
 					(unit 7)
 				)
@@
 		(dnp no)
 		(fields_autoplaced yes)
-		(property "Reference" "U15"
+		(property "Reference" "U14"
 			(at 105.41 92.71 0)
 			(effects
@@
 			(project "LiF_FC-PCB_rev1"
 				(path "/9e3e8da7-e506-46c9-90e5-307e4ad30d29/5a2c7040-8854-4895-b7b6-208daa06b69a"
-					(reference "U15")
+					(reference "U14")
 					(unit 5)
 				)
@@
 		(on_board yes)
 		(dnp no)
-		(property "Reference" "C53"
+		(property "Reference" "C47"
 			(at 25.4 162.5599 0)
 			(effects
@@
 			(project "LiF_FC-PCB_rev1"
 				(path "/9e3e8da7-e506-46c9-90e5-307e4ad30d29/5a2c7040-8854-4895-b7b6-208daa06b69a"
-					(reference "C53")
+					(reference "C47")
 					(unit 1)
 				)
@@
 		(dnp no)
 		(fields_autoplaced yes)
-		(property "Reference" "U16"
+		(property "Reference" "U15"
 			(at 105.41 125.73 0)
 			(effects
@@
 			(project "LiF_FC-PCB_rev1"
 				(path "/9e3e8da7-e506-46c9-90e5-307e4ad30d29/5a2c7040-8854-4895-b7b6-208daa06b69a"
-					(reference "U16")
+					(reference "U15")
 					(unit 1)
 				)
@@
 		(dnp no)
 		(fields_autoplaced yes)
-		(property "Reference" "U15"
+		(property "Reference" "U14"
 			(at 105.41 109.22 0)
 			(effects
@@
 			(project "LiF_FC-PCB_rev1"
 				(path "/9e3e8da7-e506-46c9-90e5-307e4ad30d29/5a2c7040-8854-4895-b7b6-208daa06b69a"
-					(reference "U15")
+					(reference "U14")
 					(unit 6)
 				)
@@
 		(on_board yes)
 		(dnp no)
-		(property "Reference" "R70"
+		(property "Reference" "R63"
 			(at 22.86 138.4299 0)
 			(effects
@@
 			(project "LiF_FC-PCB_rev1"
 				(path "/9e3e8da7-e506-46c9-90e5-307e4ad30d29/5a2c7040-8854-4895-b7b6-208daa06b69a"
-					(reference "R70")
+					(reference "R63")
 					(unit 1)
 				)
@@
 		(dnp no)
 		(fields_autoplaced yes)
-		(property "Reference" "J43"
+		(property "Reference" "J40"
 			(at 198.12 139.7 0)
 			(effects
@@
 			(project ""
 				(path "/9e3e8da7-e506-46c9-90e5-307e4ad30d29/5a2c7040-8854-4895-b7b6-208daa06b69a"
-					(reference "J43")
+					(reference "J40")
 					(unit 1)
 				)
@@
 		(on_board yes)
 		(dnp no)
-		(property "Reference" "#PWR095"
+		(property "Reference" "#PWR089"
 			(at 220.98 163.83 0)
 			(effects
@@
 			(project "LiF_FC-PCB_rev1"
 				(path "/9e3e8da7-e506-46c9-90e5-307e4ad30d29/5a2c7040-8854-4895-b7b6-208daa06b69a"
-					(reference "#PWR095")
+					(reference "#PWR089")
 					(unit 1)
 				)
@@
 		(dnp no)
 		(fields_autoplaced yes)
-		(property "Reference" "U15"
+		(property "Reference" "U14"
 			(at 105.41 63.5 0)
 			(effects
@@
 			(project "LiF_FC-PCB_rev1"
 				(path "/9e3e8da7-e506-46c9-90e5-307e4ad30d29/5a2c7040-8854-4895-b7b6-208daa06b69a"
-					(reference "U15")
+					(reference "U14")
 					(unit 3)
 				)
@@
 		(dnp no)
 		(fields_autoplaced yes)
-		(property "Reference" "U15"
+		(property "Reference" "U14"
 			(at 105.41 77.47 0)
 			(effects
@@
 			(project "LiF_FC-PCB_rev1"
 				(path "/9e3e8da7-e506-46c9-90e5-307e4ad30d29/5a2c7040-8854-4895-b7b6-208daa06b69a"
-					(reference "U15")
+					(reference "U14")
 					(unit 4)
 				)
@@
 		(on_board yes)
 		(dnp no)
-		(property "Reference" "R76"
+		(property "Reference" "R62"
 			(at 208.28 133.3499 0)
 			(effects
@@
 			(project "LiF_FC-PCB_rev1"
 				(path "/9e3e8da7-e506-46c9-90e5-307e4ad30d29/5a2c7040-8854-4895-b7b6-208daa06b69a"
-					(reference "R76")
+					(reference "R62")
 					(unit 1)
 				)
@@
 		(on_board no)
 		(dnp yes)
-		(property "Reference" "J38"
+		(property "Reference" "J39"
 			(at 42.672 45.974 90)
 			(effects
@@
 			(project "LiF_FC-PCB_rev1"
 				(path "/9e3e8da7-e506-46c9-90e5-307e4ad30d29/5a2c7040-8854-4895-b7b6-208daa06b69a"
-					(reference "J38")
+					(reference "J39")
 					(unit 1)
 				)
@@
 		(on_board yes)
 		(dnp no)
-		(property "Reference" "#PWR097"
+		(property "Reference" "#PWR087"
 			(at 255.27 119.38 0)
 			(effects
@@
 			(project "LiF_FC-PCB_rev1"
 				(path "/9e3e8da7-e506-46c9-90e5-307e4ad30d29/5a2c7040-8854-4895-b7b6-208daa06b69a"
-					(reference "#PWR097")
+					(reference "#PWR087")
 					(unit 1)
 				)
@@
 		(dnp no)
 		(fields_autoplaced yes)
-		(property "Reference" "U15"
+		(property "Reference" "U14"
 			(at 105.41 48.26 0)
 			(effects
@@
 			(project "LiF_FC-PCB_rev1"
 				(path "/9e3e8da7-e506-46c9-90e5-307e4ad30d29/5a2c7040-8854-4895-b7b6-208daa06b69a"
-					(reference "U15")
+					(reference "U14")
 					(unit 2)
 				)
@@
 		(on_board yes)
 		(dnp no)
-		(property "Reference" "#PWR0114"
+		(property "Reference" "#PWR088"
 			(at 205.74 163.83 0)
 			(effects
@@
 			(project "LiF_FC-PCB_rev1"
 				(path "/9e3e8da7-e506-46c9-90e5-307e4ad30d29/5a2c7040-8854-4895-b7b6-208daa06b69a"
-					(reference "#PWR0114")
+					(reference "#PWR088")
 					(unit 1)
 				)
@@
 		(on_board yes)
 		(dnp no)
-		(property "Reference" "C49"
+		(property "Reference" "C45"
 			(at 246.38 96.5199 0)
 			(effects
@@
 			(project "LiF_FC-PCB_rev1"
 				(path "/9e3e8da7-e506-46c9-90e5-307e4ad30d29/5a2c7040-8854-4895-b7b6-208daa06b69a"
-					(reference "C49")
+					(reference "C45")
 					(unit 1)
 				)
@@
 		(dnp no)
 		(fields_autoplaced yes)
-		(property "Reference" "#PWR098"
+		(property "Reference" "#PWR090"
 			(at 29.21 175.26 0)
 			(effects
@@
 			(project "LiF_FC-PCB_rev1"
 				(path "/9e3e8da7-e506-46c9-90e5-307e4ad30d29/5a2c7040-8854-4895-b7b6-208daa06b69a"
-					(reference "#PWR098")
+					(reference "#PWR090")
 					(unit 1)
 				)
@@
 		(on_board yes)
 		(dnp no)
-		(property "Reference" "U15"
+		(property "Reference" "U14"
 			(at 226.568 83.566 0)
 			(effects
@@
 			(project "LiF_FC-PCB_rev1"
 				(path "/9e3e8da7-e506-46c9-90e5-307e4ad30d29/5a2c7040-8854-4895-b7b6-208daa06b69a"
-					(reference "U15")
+					(reference "U14")
 					(unit 7)
 				)
@@
 		(on_board yes)
 		(dnp yes)
-		(property "Reference" "R66"
+		(property "Reference" "R61"
 			(at 40.64 58.42 90)
 			(effects
@@
 			(project "LiF_FC-PCB_rev1"
 				(path "/9e3e8da7-e506-46c9-90e5-307e4ad30d29/5a2c7040-8854-4895-b7b6-208daa06b69a"
-					(reference "R66")
+					(reference "R61")
 					(unit 1)
 				)

Commit message: progress save for the night. landmarking of service PCB is almost done. redid the analog section layout to make it more assembleable and better utilze the space. Still need to do ACC, R3V3, IO, test points, and jumpers
Connections:
- net LED0 renamed IO16
- net LED1 renamed IO17
- net LED2 renamed IO18
- net LED3 renamed IO19
- net LED4 renamed IO20
- net LED5 renamed IO21
- net LED6 renamed IO22
- net LED7 renamed IO23
Other:
- note added: "LED0"
- note added: "LED1"
- note added: "LED2"
- note added: "LED3"
- note added: "LED4"
- note added: "LED5"
- note added: "LED6"
- note added: "LED7"
Changed lines of the file:
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@@
 	(rectangle
 		(start 15.24 123.19)
-		(end 80.01 194.31)
+		(end 87.63 194.31)
 		(stroke
 			(width 0)
@@
 		)
 	)
+	(text "LED0"
+		(exclude_from_sim no)
+		(at 77.47 163.83 0)
+		(effects
+			(font
+				(size 1.27 1.27)
+			)
+			(justify right bottom)
+		)
+	)
 	(text "Lithium Firefly - Button and LED Array"
 		(exclude_from_sim no)
@@
 		)
 	)
+	(text "LED6"
+		(exclude_from_sim no)
+		(at 77.47 179.07 0)
+		(effects
+			(font
+				(size 1.27 1.27)
+			)
+			(justify right bottom)
+		)
+	)
+	(text "LED5"
+		(exclude_from_sim no)
+		(at 77.47 176.53 0)
+		(effects
+			(font
+				(size 1.27 1.27)
+			)
+			(justify right bottom)
+		)
+	)
 	(text "I2C GPIO Expander"
 		(exclude_from_sim no)
@@
 		)
 	)
+	(text "LED4"
+		(exclude_from_sim no)
+		(at 77.47 173.99 0)
+		(effects
+			(font
+				(size 1.27 1.27)
+			)
+			(justify right bottom)
+		)
+	)
+	(text "LED3"
+		(exclude_from_sim no)
+		(at 77.47 171.45 0)
+		(effects
+			(font
+				(size 1.27 1.27)
+			)
+			(justify right bottom)
+		)
+	)
+	(text "LED1"
+		(exclude_from_sim no)
+		(at 77.47 166.37 0)
+		(effects
+			(font
+				(size 1.27 1.27)
+			)
+			(justify right bottom)
+		)
+	)
 	(text "I2C addr\n0100 000x"
 		(exclude_from_sim no)
@@
 		)
 	)
+	(text "LED7"
+		(exclude_from_sim no)
+		(at 77.47 181.61 0)
+		(effects
+			(font
+				(size 1.27 1.27)
+			)
+			(justify right bottom)
+		)
+	)
 	(text "Inputs/Outputs"
 		(exclude_from_sim no)
@@
 				(bold yes)
 			)
+		)
+	)
+	(text "LED2"
+		(exclude_from_sim no)
+		(at 77.47 168.91 0)
+		(effects
+			(font
+				(size 1.27 1.27)
+			)
+			(justify right bottom)
 		)
 	)
@@
 	(wire
 		(pts
-			(xy 77.47 179.07) (xy 68.58 179.07)
+			(xy 85.09 179.07) (xy 68.58 179.07)
 		)
 		(stroke
@@
 	(wire
 		(pts
-			(xy 77.47 171.45) (xy 68.58 171.45)
+			(xy 85.09 171.45) (xy 68.58 171.45)
 		)
 		(stroke
@@
 	(wire
 		(pts
-			(xy 77.47 168.91) (xy 68.58 168.91)
+			(xy 85.09 168.91) (xy 68.58 168.91)
 		)
 		(stroke
@@
 	(wire
 		(pts
-			(xy 77.47 163.83) (xy 68.58 163.83)
+			(xy 85.09 163.83) (xy 68.58 163.83)
 		)
 		(stroke
@@
 	(wire
 		(pts
-			(xy 77.47 166.37) (xy 68.58 166.37)
+			(xy 85.09 166.37) (xy 68.58 166.37)
 		)
 		(stroke
@@
 	(wire
 		(pts
-			(xy 77.47 181.61) (xy 68.58 181.61)
+			(xy 85.09 181.61) (xy 68.58 181.61)
 		)
 		(stroke
@@
 	(wire
 		(pts
-			(xy 77.47 173.99) (xy 68.58 173.99)
+			(xy 85.09 173.99) (xy 68.58 173.99)
 		)
 		(stroke
@@
 	(wire
 		(pts
-			(xy 77.47 176.53) (xy 68.58 176.53)
+			(xy 85.09 176.53) (xy 68.58 176.53)
 		)
 		(stroke
@@
 		(pts
 			(xy 260.35 110.49) (xy 260.35 111.76)
+		)
+		(stroke
+			(width 0)
+			(type default)
+		)
+	)
+	(bus
+		(pts
+			(xy 34.29 116.84) (xy 60.96 116.84)
 		)
 		(stroke
@@
 		)
 	)
-	(label "LED5"
-		(at 77.47 176.53 180)
-		(effects
-			(font
-				(size 1.27 1.27)
-			)
-			(justify right bottom)
-		)
-	)
 	(label "BTN0"
 		(at 77.47 140.97 180)
@@
 		)
 	)
-	(label "LED0"
-		(at 77.47 163.83 180)
-		(effects
-			(font
-				(size 1.27 1.27)
-			)
-			(justify right bottom)
-		)
-	)
 	(label "BTN7"
 		(at 77.47 158.75 180)
@@
 		)
 	)
+	(label "IO23"
+		(at 85.09 181.61 180)
+		(effects
+			(font
+				(size 1.27 1.27)
+			)
+			(justify right bottom)
+		)
+	)
 	(label "I2C.SCL"
 		(at 31.75 140.97 0)
@@
 		)
 	)
+	(label "IO19"
+		(at 85.09 171.45 180)
+		(effects
+			(font
+				(size 1.27 1.27)
+			)
+			(justify right bottom)
+		)
+	)
 	(label "~{BTN_IRQ}"
 		(at 31.75 148.59 0)
@@
 		)
 	)
-	(label "LED3"
-		(at 77.47 171.45 180)
-		(effects
-			(font
-				(size 1.27 1.27)
-			)
-			(justify right bottom)
-		)
-	)
 	(label "IN6"
 		(at 119.38 134.62 180)
@@
 		)
 	)
-	(label "LED2"
-		(at 77.47 168.91 180)
-		(effects
-			(font
-				(size 1.27 1.27)
-			)
-			(justify right bottom)
-		)
-	)
-	(label "LED6"
-		(at 77.47 179.07 180)
-		(effects
-			(font
-				(size 1.27 1.27)
-			)
-			(justify right bottom)
-		)
-	)
 	(label "~{BTN_IRQ}"
 		(at 60.96 100.33 180)
@@
 		)
 	)
-	(label "LED4"
-		(at 77.47 173.99 180)
+	(label "IO17"
+		(at 85.09 166.37 180)
+		(effects
+			(font
+				(size 1.27 1.27)
+			)
+			(justify right bottom)
+		)
+	)
+	(label "IO18"
+		(at 85.09 168.91 180)
+		(effects
+			(font
+				(size 1.27 1.27)
+			)
+			(justify right bottom)
+		)
+	)
+	(label "IO22"
+		(at 85.09 179.07 180)
 		(effects
 			(font
@@
 		)
 	)
+	(label "IO21"
+		(at 85.09 176.53 180)
+		(effects
+			(font
+				(size 1.27 1.27)
+			)
+			(justify right bottom)
+		)
+	)
 	(label "I2C.SDA"
 		(at 31.75 143.51 0)
@@
 		)
 	)
-	(label "LED7"
-		(at 77.47 181.61 180)
-		(effects
-			(font
-				(size 1.27 1.27)
-			)
-			(justify right bottom)
-		)
-	)
-	(label "LED1"
-		(at 77.47 166.37 180)
+	(label "IO20"
+		(at 85.09 173.99 180)
 		(effects
 			(font
@@
 		)
 	)
+	(label "IO16"
+		(at 85.09 163.83 180)
+		(effects
+			(font
+				(size 1.27 1.27)
+			)
+			(justify right bottom)
+		)
+	)
 	(label "BTN5"
 		(at 92.71 118.11 0)
@@
 	(label "BTN2"
 		(at 77.47 146.05 180)
+		(effects
+			(font
+				(size 1.27 1.27)
+			)
+			(justify right bottom)
+		)
+	)
+	(label "IO[16..23]"
+		(at 60.96 116.84 180)
 		(effects
 			(font
@@
 		(effects
 			(font
+				(size 1.27 1.27)
+			)
+			(justify right)
+		)
+	)
+	(hierarchical_label "IO[16..23]"
+		(shape bidirectional)
+		(at 34.29 116.84 180)
+		(effects
+			(font
