File: KiCAD/LiF_FC-PCB_rev1/LiF_FC-PCB_rev1.kicad_pcb (KiCad board)
At the start: 4 copper layers, 86.5 x 61 mm, 279 parts, among them J1 VCAN_{EN}, J10 R3V3_{EN}, J11 A3V3_{EN}, J12 ESP 3V3_{EN}, J13 ESP_DGB_CONN, J14 CAN Upstream, J15 ESP_DGB_CONN, J16 ESP_DGB_CONN, J17 LC 5V0_{EN}, J18 LC 3V3_{EN}, J19 Load Cell, J2 R5V0_{EN}, J20 Bypass DOWN fuse, J21 CAN Down_{EN}, J22 CAN Upstream, J23 CAN 5V0_{EN}, J24 Bypass OR-ing, J25 Bypass DOWN fuse, J26 CAN 3V3_{EN}, J27 CAN UP_{EN}, J28 CAN Downstream, J29 Use DB9 VBUS, J3 REG V_{IN} EN, J30 DE9_Socket_MountingHoles, J31 ACC 3V3_{EN}, J32 Amp V select, J33 ST 1 Bypass, J34 ST 2 Bypass, J35 Vol Pot Bypass, J36 SKP OUT, J37 BTN 3V3_{EN}, J38 BTN 3V3_{EN}, J39 ENC 3V3_{EN}, J4 Barrel Jack, J40 SRV 3V3_{EN}, J41 Servo A, J42 Servo B, J43 Door Closed, J5 CAN USB_{EN}, J6 PROG USB_{EN}, J7 V_{IN}, J8 3V3 REG_{EN}, J9 A3V3 REG_{EN}, Q1 MMBT4401, Q2 MMBT4401, SW1 Flash, SW10 TL3301PF160QG, SW11 TL3301PF160QG, SW2 Reset, SW3 CAN Termination Select, SW4 TL3301PF160QG, SW5 TL3301PF160QG, SW6 TL3301PF160QG, SW7 TL3301PF160QG, SW8 TL3301PF160QG, SW9 TL3301PF160QG, U1 AZ1117-3.3, U10 MCP2542FD-E/SN, U11 BMA400, U12 PAM8302AAS, U13 DC56-11EWA, U14 NCA9555, U15 SN74HC14DR, U16 SN74HC14DR, U17 NCA9555, U2 AZ1117-3.3, U3 TPS2117DRLR, U4 TPS2117DRLR, U5 LMR14050, U6 ESP32-S3-WROOM-1, U7 CY7C65213-28PVXI, U8 MCP6N11-xxxE/SN, U9 NCV8114ASN165T1G

Commit message: backup before expanding the board size
Parts:
- removed D1: D, Diode_SMD:D_SOD-123F
- removed J30: DE9_Socket_MountingHoles, LiF_PCB_Footprints:CONN_DB-9 Female KG-T4S_ASM
- removed J4: Barrel Jack, Connector_BarrelJack:BarrelJack_GCT_DCJ200-10-A_Horizontal
- removed JP1: BTN3, Jumper:SolderJumper-2_P1.3mm_Open_RoundedPad1.0x1.5mm
- removed JP2: BTN4, Jumper:SolderJumper-2_P1.3mm_Open_RoundedPad1.0x1.5mm
- removed JP3: BTN5, Jumper:SolderJumper-2_P1.3mm_Open_RoundedPad1.0x1.5mm
- added J44: CAN, Connector_JST:JST_PH_B4B-PH-K_1x04_P2.00mm_Vertical, F.Cu at (147.6, 61.5)
- C43, C44, C45, C46, C47, C50, C51, C52, D16, D17, D18, D19, D20, D21, D22, D23, R61, R62, R63, R64, R65, R67, R68, R69, SW10, SW11, SW4, SW5, SW6, SW7, SW8, SW9, U13: moved to B.Cu
- SW1, SW2: footprint LiF_PCB_Footprints:SW_TL3301PF160QG -> LiF_PCB_Footprints:SON4_PTS526 SM15 SMTR2 LFS_CNK
- SW3: value CAN Termination Select -> CAN Termination; footprint LiF_PCB_Footprints:SW_SLW-883935-2A-D -> LiF_PCB_Footprints:SW_JS202011JCQN
- TP16, TP20: value GND -> GNDA
- TP18: value FLT -> LC_FLT
- moved TP24 311.5 mm to (193.0, 84.0)
- moved C33 267.2 mm to (145.0, 71.8), turned to -90 degrees
- moved R53 265.6 mm to (142.2, 66.8), turned to 180 degrees
- moved C34 264.7 mm to (142.5, 78.0)
- moved TP22 252.3 mm to (132.0, 61.0)
- moved U10 252.0 mm to (141.0, 73.0), turned to 90 degrees
- moved J15 250.3 mm to (132.0, 103.0), turned to -90 degrees
- moved TP23 248.9 mm to (128.0, 61.0)
- moved U6 243.1 mm to (125.0, 118.5), turned to 180 degrees
- moved J13 241.9 mm to (136.5, 123.8), turned to 180 degrees
- moved SW3 239.4 mm to (137.0, 64.0)
- moved D15 237.3 mm to (142.2, 62.2), turned to -90 degrees
- moved J28 229.0 mm to (144.5, 53.0), turned to 180 degrees
- moved J14 228.7 mm to (142.5, 122.0)
- moved J22 216.7 mm to (133.5, 53.0), turned to 180 degrees
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Connections:
- R53 pad 2: Net-(SW3-C) -> Net-(SW3B-C)
- RN1 pad 1: /Display/DIG1_A -> /Display/DIG1_DP
- RN1 pad 10: Net-(U13-DIG1_G) -> Net-(U13-DIG1_B)
- RN1 pad 11: Net-(U13-DIG1_F) -> Net-(U13-DIG1_C)
- RN1 pad 12: Net-(U13-DIG1_E) -> Net-(U13-DIG1_D)
- RN1 pad 13: Net-(U13-DIG1_D) -> Net-(U13-DIG1_E)
- RN1 pad 14: Net-(U13-DIG1_C) -> Net-(U13-DIG1_F)
- RN1 pad 15: Net-(U13-DIG1_B) -> Net-(U13-DIG1_G)
- RN1 pad 16: Net-(U13-DIG1_A) -> Net-(U13-DP1)
- RN1 pad 2: /Display/DIG1_B -> /Display/DIG1_G
- RN1 pad 3: /Display/DIG1_C -> /Display/DIG1_F
- RN1 pad 4: /Display/DIG1_D -> /Display/DIG1_E
- RN1 pad 5: /Display/DIG1_E -> /Display/DIG1_D
- RN1 pad 6: unconnected-(RN1-Pad6) -> /Display/DIG1_C
- RN1 pad 7: /Display/DIG1_G -> /Display/DIG1_B
- RN1 pad 8: /Display/DIG1_DP -> /Display/DIG1_A
- RN1 pad 9: Net-(U13-DP1) -> Net-(U13-DIG1_A)
- RN2 pad 1: /Display/DIG2_A -> /Display/DIG2_DP
- RN2 pad 10: Net-(U13-DIG2_G) -> Net-(U13-DIG2_B)
- RN2 pad 11: Net-(U13-DIG2_F) -> Net-(U13-DIG2_C)
- RN2 pad 12: Net-(U13-DIG2_E) -> Net-(U13-DIG2_D)
- RN2 pad 13: Net-(U13-DIG2_D) -> Net-(U13-DIG2_E)
- RN2 pad 14: Net-(U13-DIG2_C) -> Net-(U13-DIG2_F)
- RN2 pad 15: Net-(U13-DIG2_B) -> Net-(U13-DIG2_G)
- RN2 pad 16: Net-(U13-DIG2_A) -> Net-(U13-DP2)
- RN2 pad 2: /Display/DIG2_B -> /Display/DIG2_G
- RN2 pad 3: /Display/DIG2_C -> /Display/DIG2_F
- RN2 pad 4: /Display/DIG2_D -> /Display/DIG2_E
- RN2 pad 5: /Display/DIG2_E -> /Display/DIG2_D
- RN2 pad 6: unconnected-(RN2-Pad6) -> /Display/DIG2_C
- RN2 pad 7: /Display/DIG2_G -> /Display/DIG2_B
- RN2 pad 8: /Display/DIG2_DP -> /Display/DIG2_A
- RN2 pad 9: Net-(U13-DP2) -> Net-(U13-DIG2_A)
- SW3 pad 2: /CAN/CAN+ -> unconnected-(SW3A-B-Pad2)
- SW3 pad 3: Net-(SW3-C) -> unconnected-(SW3A-C-Pad3)
- U14 pad 18: unconnected-(U14-IO1_5-Pad18) -> /Display/DIG2_F
- U14 pad 9: unconnected-(U14-IO0_5-Pad9) -> /Display/DIG1_F
- U15 pad 10: Net-(JP2-B) -> /Buttons/BTN4
- U15 pad 12: Net-(JP3-A) -> /Buttons/BTN5
- U15 pad 8: Net-(JP1-A) -> /Buttons/BTN3
Routing:
- net /CAN/CAN+: track 0.00 -> 50.1 mm, vias 0 -> 3
- net /CAN/CAN-: track 0.00 -> 43.4 mm
- net Net-(SW3B-C): track 0.00 -> 5.23 mm
- net /CAN/CAN_5V0: track 0.00 -> 2.56 mm
- net /CAN/CAN_3V3: track 0.00 -> 2.21 mm
- net GND: track 0.00 -> 1.19 mm, vias 0 -> 1
Other:
- board size 86.5 x 61 mm -> 50 x 85 mm

Commit message: backup before leaving school
Parts:
- J1, J10, J11, J12, J17, J18, J2, J20, J21, J23, J24, J25, J26, J27, J29, J3, J31, J33, J34, J35, J37, J38, J39, J40, J5, J6, J8, J9: footprint Connector_PinHeader_2.54mm:PinHeader_1x02_P2.54mm_Vertical -> Connector_PinHeader_2.54mm:PinHeader_1x02_P2.54mm_Vertical_SMD_Pin1Left
- J32: footprint Connector_PinHeader_2.54mm:PinHeader_1x03_P2.54mm_Vertical -> Connector_PinHeader_2.54mm:PinHeader_1x03_P2.54mm_Vertical_SMD_Pin1Left
- moved R52 52.8 mm to (90.0, 44.5), turned to 180 degrees
- moved R49 43.3 mm to (80.0, 44.5)
- moved J13 42.7 mm to (152.2, 84.1), turned to -90 degrees
- moved R47 32.6 mm to (66.5, 46.0), turned to 180 degrees
- moved U6 31.7 mm to (147.0, 95.6), turned to -90 degrees
- moved TP22 24.4 mm to (154.0, 50.5)
- moved R43 23.7 mm to (60.0, 32.5)
- moved TP23 22.1 mm to (147.5, 50.5)
- moved J16 22.1 mm to (135.6, 107.1), turned to 90 degrees
- moved C52 21.6 mm to (118.0, 110.5)
- moved D23 21.6 mm to (122.0, 110.5)
- moved R69 21.6 mm to (126.0, 110.5)
- moved SW11 21.6 mm to (122.0, 115.0)
- moved C43 17.2 mm to (104.0, 50.5)
- moved C44 17.2 mm to (118.0, 50.5)
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Routing:
- net /CAN/CAN-: track 43.4 -> 52.8 mm, vias 0 -> 2
- net /CAN/CAN+: track 50.1 -> 47.5 mm, vias 3 -> 1
- net Net-(SW3B-C): track 5.23 -> 6.71 mm
Other:
- board size 50 x 85 mm -> 60 x 100 mm
- board text added: "1 2"
- board text added: "3 4"
- board text added: "5 6"
- board text added: "door call"

Commit message: progress backup before increasing the size of the PCB again
Parts:
- removed J2: R5V0_{EN}, Connector_PinHeader_2.54mm:PinHeader_1x02_P2.54mm_Vertical_SMD_Pin1Left
- removed J20, J25: Bypass DOWN fuse, Connector_PinHeader_2.54mm:PinHeader_1x02_P2.54mm_Vertical_SMD_Pin1Left
- removed J21: CAN Down_{EN}, Connector_PinHeader_2.54mm:PinHeader_1x02_P2.54mm_Vertical_SMD_Pin1Left
- removed J23: CAN 5V0_{EN}, Connector_PinHeader_2.54mm:PinHeader_1x02_P2.54mm_Vertical_SMD_Pin1Left
- removed J24: Bypass OR-ing, Connector_PinHeader_2.54mm:PinHeader_1x02_P2.54mm_Vertical_SMD_Pin1Left
- removed J26: CAN 3V3_{EN}, Connector_PinHeader_2.54mm:PinHeader_1x02_P2.54mm_Vertical_SMD_Pin1Left
- removed J27: CAN UP_{EN}, Connector_PinHeader_2.54mm:PinHeader_1x02_P2.54mm_Vertical_SMD_Pin1Left
- removed J29: Use DB9 VBUS, Connector_PinHeader_2.54mm:PinHeader_1x02_P2.54mm_Vertical_SMD_Pin1Left
- removed J3: REG V_{IN} EN, Connector_PinHeader_2.54mm:PinHeader_1x02_P2.54mm_Vertical_SMD_Pin1Left
- removed J32: Amp V select, Connector_PinHeader_2.54mm:PinHeader_1x03_P2.54mm_Vertical_SMD_Pin1Left
- removed J33: ST 1 Bypass, Connector_PinHeader_2.54mm:PinHeader_1x02_P2.54mm_Vertical_SMD_Pin1Left
- removed J34: ST 2 Bypass, Connector_PinHeader_2.54mm:PinHeader_1x02_P2.54mm_Vertical_SMD_Pin1Left
- removed J35: Vol Pot Bypass, Connector_PinHeader_2.54mm:PinHeader_1x02_P2.54mm_Vertical_SMD_Pin1Left
- removed J38: BTN 3V3_{EN}, Connector_PinHeader_2.54mm:PinHeader_1x02_P2.54mm_Vertical_SMD_Pin1Left
- removed J39: ENC 3V3_{EN}, Connector_PinHeader_2.54mm:PinHeader_1x02_P2.54mm_Vertical_SMD_Pin1Left
- removed J5: CAN USB_{EN}, Connector_PinHeader_2.54mm:PinHeader_1x02_P2.54mm_Vertical_SMD_Pin1Left
- removed R3: 0, Resistor_SMD:R_0805_2012Metric
- added H1: MountingHole, MountingHole:MountingHole_3.2mm_M3_DIN965, F.Cu at (115.0, 56.5)
- added H2: MountingHole, MountingHole:MountingHole_3.2mm_M3_DIN965, F.Cu at (105.0, 117.5)
- added H3: MountingHole, MountingHole:MountingHole_3.2mm_M3_DIN965, F.Cu at (155.0, 117.5)
- added J45: Conn_01x10_Socket, Connector_PinHeader_2.54mm:PinHeader_1x10_P2.54mm_Vertical, F.Cu at (133.6, 36.8)
- added J46: Conn_01x22_Socket, Connector_PinHeader_2.54mm:PinHeader_1x22_P2.54mm_Vertical, F.Cu at (103.3, 123.2)
- added J47: Conn_01x16_Pin, Connector_PinHeader_2.54mm:PinHeader_1x16_P2.54mm_Vertical, F.Cu at (111.0, 120.7)
- J13, J15, J16, J19, J44, J7, R2, R4, R43, R47, R49, R52, TP10, TP11, TP15, TP16, TP17, TP18, TP19, TP21, TP7: moved to B.Cu
- moved R26 344.4 mm to (219.2, 17.0), turned to 180 degrees
- moved R27 343.4 mm to (219.2, 28.2), turned to 180 degrees
- moved U7 318.3 mm to (228.0, 21.0), turned to -90 degrees
- moved F2 312.9 mm to (219.2, 26.0)
- moved C24 312.3 mm to (180.2, 131.6)
- moved R29 311.9 mm to (184.3, 131.3)
- moved R32 311.5 mm to (183.4, 142.2), turned to 90 degrees
- moved R33 309.7 mm to (183.4, 137.8), turned to -90 degrees
- moved C22 306.8 mm to (172.8, 132.2)
- moved C23 306.8 mm to (172.8, 135.2)
- moved R28 306.8 mm to (177.2, 135.2)
- moved R30 303.8 mm to (179.1, 121.4)
- moved R31 303.8 mm to (179.1, 124.4)
- moved D12 297.9 mm to (219.2, 21.5), turned to 180 degrees
- moved D11 297.8 mm to (219.2, 19.2), turned to 180 degrees
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Connections:
- net /MCU/D+ renamed /MCU/USB.D+
- net /MCU/D- renamed /MCU/USB.D-
- D2 pad 1: Net-(D2-K) -> /Power Regulation/5V Regulator/REG5V_in
- J7 pad 1: /Power Regulation/V_{supply} -> GND
- J7 pad 2: GND -> /Power Regulation/V_{supply}
- U6 pad 36: /MCU/ESP32_37 -> /MCU/ESP32_36
- U6 pad 37: /MCU/ESP32_36 -> /MCU/ESP32_37
- U7 pad 1: /MCU/ESP32_37 -> /MCU/ESP32_36
- U7 pad 5: /MCU/ESP32_36 -> /MCU/ESP32_37
Routing:
- net /MCU/USB.D+: track 0.00 -> 14.1 mm
- net /MCU/USB.D-: track 0.00 -> 13.2 mm
- net /CAN/CAN+: track 47.5 -> 48.5 mm
- net /CAN/CAN-: track 52.8 -> 51.9 mm
Other:
- board size 60 x 100 mm -> 155 x 90 mm

Commit message: looks like I found a good layout. Need to finish landmarking and start actually routing
Parts:
- added J47: Conn_01x16_Pin, Connector_PinHeader_2.54mm:PinHeader_1x16_P2.54mm_Vertical, F.Cu at (102.0, 111.1)
- J36, J41, J42, J43: moved to B.Cu
- moved C33 464.3 mm to (-310.0, 361.8)
- moved C34 464.3 mm to (-312.5, 368.0)
- moved C43 464.3 mm to (-359.0, 349.0)
- moved C44 464.3 mm to (-345.0, 349.0)
- moved C45 464.3 mm to (-359.0, 368.5)
- moved C46 464.3 mm to (-345.0, 368.5)
- moved C47 464.3 mm to (-359.0, 389.0)
- moved C48 464.3 mm to (-306.8, 411.5)
- moved C49 464.3 mm to (-315.2, 411.5)
- moved C50 464.3 mm to (-345.0, 389.0)
- moved C51 464.3 mm to (-359.0, 409.0)
- moved C52 464.3 mm to (-345.0, 409.0)
- moved D15 464.3 mm to (-312.8, 352.2)
- moved D16 464.3 mm to (-355.0, 389.0)
- moved D17 464.3 mm to (-341.0, 389.0)
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Routing:
- net /CAN/CAN+: track 48.5 -> 62.9 mm
- net /CAN/CAN-: track 51.9 -> 65.9 mm
Other:
- board size 155 x 90 mm -> 197.2 x 94.8 mm

Commit message: backup before splitting the schematics into 2 boards: I/O PCB and Service PCB
Parts:
- removed JP4: ENC SW, Jumper:SolderJumper-2_P1.3mm_Open_RoundedPad1.0x1.5mm
- removed JP5: ENC A, Jumper:SolderJumper-2_P1.3mm_Open_RoundedPad1.0x1.5mm
- removed JP6: ENC B, Jumper:SolderJumper-2_P1.3mm_Open_RoundedPad1.0x1.5mm
- RV1, SW1, SW2: moved to B.Cu
- moved U15 552.6 mm to (124.8, 74.8), turned to 90 degrees
- moved C48 543.9 mm to (118.8, 72.8), turned to -90 degrees
- moved C49 543.2 mm to (110.8, 74.5)
- moved U16 543.2 mm to (108.8, 80.5)
- moved SW2 263.8 mm to (153.0, 121.0)
- moved TP28 262.2 mm to (128.8, 67.2), turned to 90 degrees
- moved SW1 257.6 mm to (145.0, 120.2), turned to 90 degrees
- moved R50 253.4 mm to (129.5, 56.2), turned to 90 degrees
- moved R51 251.5 mm to (127.2, 56.2), turned to 90 degrees
- moved C58 247.6 mm to (119.0, 60.8), turned to 90 degrees
- moved C39 243.2 mm to (116.8, 60.8), turned to 90 degrees
- moved C40 242.7 mm to (116.8, 65.9), turned to 90 degrees
- moved R57 241.5 mm to (119.0, 65.9), turned to -90 degrees
- moved C41 239.0 mm to (112.2, 65.9), turned to -90 degrees
- moved R58 237.8 mm to (114.5, 65.9), turned to 90 degrees
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- renumbered C06_1 to C58
Routing:
- net unconnected-(J47-Pin_1-Pad1): track 0.00 -> 21.9 mm
- net unconnected-(J47-Pin_2-Pad2): track 0.00 -> 19.3 mm
- net unconnected-(J47-Pin_3-Pad3): track 0.00 -> 16.5 mm
- net unconnected-(J47-Pin_4-Pad4): track 0.00 -> 14.3 mm
- net unconnected-(J47-Pin_5-Pad5): track 0.00 -> 10.7 mm
- net unconnected-(J47-Pin_6-Pad6): track 0.00 -> 8.02 mm
- net unconnected-(J47-Pin_7-Pad7): track 0.00 -> 5.15 mm
- net /MCU/USB.D-: track 13.2 -> 15.2 mm
- net /MCU/USB.D+: track 14.1 -> 13.1 mm
Other:
- board size 197.2 x 94.8 mm -> 205 x 104.8 mm
- board text added: "DOWN"
- board text added: "UP"

Commit message: Created new KiCAD project for IO PCB, moved relevant components there, saving backup before reannotating the Service PCB schematics
Parts:
- removed C43, C44, C45, C46, C47, C50, C51, C52: 1u, Capacitor_SMD:C_0805_2012Metric
- removed C54, C55, C56: 0.1u, Capacitor_SMD:C_0805_2012Metric
- removed D16: LED0, LED_SMD:LED_0805_2012Metric
- removed D17: LED1, LED_SMD:LED_0805_2012Metric
- removed D18: LED2, LED_SMD:LED_0805_2012Metric
- removed D19: LED3, LED_SMD:LED_0805_2012Metric
- removed D20: LED4, LED_SMD:LED_0805_2012Metric
- removed D21: LED5, LED_SMD:LED_0805_2012Metric
- removed D22: LED6, LED_SMD:LED_0805_2012Metric
- removed D23: LED7, LED_SMD:LED_0805_2012Metric
- removed J1: VCAN_{EN}, Connector_PinHeader_2.54mm:PinHeader_1x02_P2.54mm_Vertical_SMD_Pin1Left
- removed J10: R3V3_{EN}, Connector_PinHeader_2.54mm:PinHeader_1x02_P2.54mm_Vertical_SMD_Pin1Left
- removed J11: A3V3_{EN}, Connector_PinHeader_2.54mm:PinHeader_1x02_P2.54mm_Vertical_SMD_Pin1Left
- removed J12: ESP 3V3_{EN}, Connector_PinHeader_2.54mm:PinHeader_1x02_P2.54mm_Vertical_SMD_Pin1Left
- removed J17: LC 5V0_{EN}, Connector_PinHeader_2.54mm:PinHeader_1x02_P2.54mm_Vertical_SMD_Pin1Left
- removed J18: LC 3V3_{EN}, Connector_PinHeader_2.54mm:PinHeader_1x02_P2.54mm_Vertical_SMD_Pin1Left
- removed J31: ACC 3V3_{EN}, Connector_PinHeader_2.54mm:PinHeader_1x02_P2.54mm_Vertical_SMD_Pin1Left
- removed J37: BTN 3V3_{EN}, Connector_PinHeader_2.54mm:PinHeader_1x02_P2.54mm_Vertical_SMD_Pin1Left
- removed J40: SRV 3V3_{EN}, Connector_PinHeader_2.54mm:PinHeader_1x02_P2.54mm_Vertical_SMD_Pin1Left
- removed J46: Conn_01x22_Socket, Connector_PinHeader_2.54mm:PinHeader_1x22_P2.54mm_Vertical
- removed J6: PROG USB_{EN}, Connector_PinHeader_2.54mm:PinHeader_1x02_P2.54mm_Vertical_SMD_Pin1Left
- removed J8: 3V3 REG_{EN}, Connector_PinHeader_2.54mm:PinHeader_1x02_P2.54mm_Vertical_SMD_Pin1Left
- removed J9: A3V3 REG_{EN}, Connector_PinHeader_2.54mm:PinHeader_1x02_P2.54mm_Vertical_SMD_Pin1Left
- removed MT1: PEC11R-4215F-S0024, LiF_PCB_Footprints:XDCR_PEC11R-4215F-S0024
- removed R61, R62, R63, R64, R65, R67, R68, R69, R71, R73, R74: 10k, Resistor_SMD:R_0805_2012Metric
- removed RN1, RN2, RN3: 8x 470, LiF_PCB_Footprints:RESCAXE50P380X160X55-16N
- removed SW10, SW11, SW4, SW5, SW6, SW7, SW8, SW9: TL3301PF160QG, LiF_PCB_Footprints:SW_TL3301PF160QG
- removed U13: DC56-11EWA, Display_7Segment:DA56-11SURKWA
- added J48: Conn_01x16_Pin, Connector_PinHeader_2.54mm:PinHeader_1x16_P2.54mm_Vertical, F.Cu at (46.8, 58.9)
Connections:
- F1 pad 2: /SYS5V0 -> /R3V3
- J45 pad 1: unconnected-(J45-Pin_1-Pad1) -> /R3V3
- J47 pad 1: (no net) -> /Display/IO0
- J47 pad 10: (no net) -> /Display/IO9
- J47 pad 11: (no net) -> /Display/IO10
- J47 pad 12: (no net) -> /Display/IO11
- J47 pad 13: (no net) -> /Display/IO12
- J47 pad 14: (no net) -> /Display/IO13
- J47 pad 15: (no net) -> /Display/IO14
- J47 pad 16: (no net) -> /Display/IO15
- J47 pad 2: (no net) -> /Display/IO1
- J47 pad 3: (no net) -> /Display/IO2
- J47 pad 4: (no net) -> /Display/IO3
- J47 pad 5: (no net) -> /Display/IO4
- J47 pad 6: (no net) -> /Display/IO5
- J47 pad 7: (no net) -> /Display/IO6
- J47 pad 8: (no net) -> /Display/IO7
- J47 pad 9: (no net) -> /Display/IO8
- J47 pad 1: unconnected-(J47-Pin_1-Pad1) -> /Display/IO0
- J47 pad 10: unconnected-(J47-Pin_10-Pad10) -> /Display/IO9
- J47 pad 11: unconnected-(J47-Pin_11-Pad11) -> /Display/IO10
- J47 pad 12: unconnected-(J47-Pin_12-Pad12) -> /Display/IO11
- J47 pad 13: unconnected-(J47-Pin_13-Pad13) -> /Display/IO12
- J47 pad 14: unconnected-(J47-Pin_14-Pad14) -> /Display/IO13
- J47 pad 15: unconnected-(J47-Pin_15-Pad15) -> /Display/IO14
- J47 pad 16: unconnected-(J47-Pin_16-Pad16) -> /Display/IO15
- J47 pad 2: unconnected-(J47-Pin_2-Pad2) -> /Display/IO1
- J47 pad 3: unconnected-(J47-Pin_3-Pad3) -> /Display/IO2
- J47 pad 4: unconnected-(J47-Pin_4-Pad4) -> /Display/IO3
- J47 pad 5: unconnected-(J47-Pin_5-Pad5) -> /Display/IO4
- J47 pad 6: unconnected-(J47-Pin_6-Pad6) -> /Display/IO5
- J47 pad 7: unconnected-(J47-Pin_7-Pad7) -> /Display/IO6
- J47 pad 8: unconnected-(J47-Pin_8-Pad8) -> /Display/IO7
- J47 pad 9: unconnected-(J47-Pin_9-Pad9) -> /Display/IO8
- R35 pad 2: /SYS5V0 -> /R3V3
- R46 pad 2: /SYS5V0 -> /R3V3
- R56 pad 2: /SYS5V0 -> /R3V3
- R6 pad 2: /SYS5V0 -> /R3V3
- R7 pad 2: /SYS5V0 -> /R3V3
- R75 pad 2: /SYS5V0 -> /R3V3
- TP2 pad 1: /SYS5V0 -> /R3V3
- U14 pad 10: /Display/DIG1_G -> /Display/IO6
- U14 pad 11: /Display/DIG1_DP -> /Display/IO7
- U14 pad 13: /Display/DIG2_A -> /Display/IO8
- U14 pad 14: /Display/DIG2_B -> /Display/IO9
- U14 pad 15: /Display/DIG2_C -> /Display/IO10
- U14 pad 16: /Display/DIG2_D -> /Display/IO11
- U14 pad 17: /Display/DIG2_E -> /Display/IO12
- U14 pad 18: /Display/DIG2_F -> /Display/IO13
- U14 pad 19: /Display/DIG2_G -> /Display/IO14
- U14 pad 20: /Display/DIG2_DP -> /Display/IO15
- U14 pad 4: /Display/DIG1_A -> /Display/IO0
- U14 pad 5: /Display/DIG1_B -> /Display/IO1
- U14 pad 6: /Display/DIG1_C -> /Display/IO2
- U14 pad 7: /Display/DIG1_D -> /Display/IO3
- U14 pad 8: /Display/DIG1_E -> /Display/IO4
- U14 pad 9: /Display/DIG1_F -> /Display/IO5
- U15 pad 1: Net-(C43-Pad1) -> /Buttons/IN0
- U15 pad 11: Net-(C47-Pad1) -> /Buttons/IN4
- U15 pad 13: Net-(C50-Pad1) -> /Buttons/IN5
- U15 pad 3: Net-(C44-Pad1) -> /Buttons/IN1
- U15 pad 5: Net-(C45-Pad1) -> /Buttons/IN2
- U15 pad 9: Net-(C46-Pad1) -> /Buttons/IN3
- U16 pad 1: Net-(C51-Pad1) -> /Buttons/IN6
- U16 pad 10: Net-(JP6-A) -> /Encoder/ENC.B
- U16 pad 11: Net-(C56-Pad1) -> /Encoder/IN10
- U16 pad 3: Net-(C52-Pad1) -> /Buttons/IN7
- U16 pad 5: Net-(C54-Pad1) -> /Encoder/IN8
- U16 pad 6: Net-(JP4-A) -> /Encoder/ENC.SW
- U16 pad 8: Net-(JP5-A) -> /Encoder/ENC.A
- U16 pad 9: Net-(C55-Pad1) -> /Encoder/IN9
Routing:
- net unconnected-(J47-Pin_1-Pad1): track 21.9 -> 0.00 mm
- net /Display/IO0: track 0.00 -> 21.9 mm
- net unconnected-(J47-Pin_2-Pad2): track 19.3 -> 0.00 mm
- net /Display/IO1: track 0.00 -> 19.3 mm
- net unconnected-(J47-Pin_3-Pad3): track 16.5 -> 0.00 mm
- net /Display/IO2: track 0.00 -> 16.5 mm
- net unconnected-(J47-Pin_4-Pad4): track 14.3 -> 0.00 mm
- net /Display/IO3: track 0.00 -> 14.3 mm
- net unconnected-(J47-Pin_5-Pad5): track 10.7 -> 0.00 mm
- net /Display/IO4: track 0.00 -> 10.7 mm
- net unconnected-(J47-Pin_6-Pad6): track 8.02 -> 0.00 mm
- net /Display/IO5: track 0.00 -> 8.02 mm
- net unconnected-(J47-Pin_7-Pad7): track 5.15 -> 0.00 mm
- net /Display/IO6: track 0.00 -> 5.15 mm
