File: KiCAD/LiF_FC-PCB_rev1/LiF_FC-PCB_rev1.kicad_pcb (KiCad board)
At the start: 4 copper layers, 205 x 104.8 mm, 205 parts, among them J13 ESP_DGB_CONN, J14 CAN Upstream, J15 ESP_DGB_CONN, J16 ESP_DGB_CONN, J19 Load Cell, J22 CAN Upstream, J28 CAN Downstream, J36 SKP OUT, J41 Servo A, J42 Servo B, J43 Door Closed, J44 CAN, J45 Conn_01x10_Socket, J47 Conn_01x16_Pin, J48 Conn_01x16_Pin, J7 V_{IN}, Q1 MMBT4401, Q2 MMBT4401, SW1 Flash, SW2 Reset, SW3 CAN Termination, U1 AZ1117-3.3, U10 MCP2542FD-E/SN, U11 BMA400, U12 PAM8302AAS, U14 NCA9555, U15 SN74HC14DR, U16 SN74HC14DR, U17 NCA9555, U2 AZ1117-3.3, U3 TPS2117DRLR, U4 TPS2117DRLR, U5 LMR14050, U6 ESP32-S3-WROOM-1, U7 CY7C65213-28PVXI, U8 MCP6N11-xxxE/SN, U9 NCV8114ASN165T1G

Commit message: backup before redoing the analog section
Parts:
- removed C48, C49, C53, C58: 0.1u, Capacitor_SMD:C_0805_2012Metric
- removed C57: 1u, Capacitor_SMD:C_0805_2012Metric
- removed J36: SKP OUT, Connector_JST:JST_PH_B2B-PH-K_1x02_P2.00mm_Vertical
- removed J41: Servo A, Connector_JST:JST_PH_B3B-PH-K_1x03_P2.00mm_Vertical
- removed J42: Servo B, Connector_JST:JST_PH_B3B-PH-K_1x03_P2.00mm_Vertical
- removed the J47 at (168.0, 111.1)
- removed J48: Conn_01x16_Pin, Connector_PinHeader_2.54mm:PinHeader_1x16_P2.54mm_Vertical
- removed R70, R76: 10k, Resistor_SMD:R_0805_2012Metric
- removed R72, R75: 0, Resistor_SMD:R_0805_2012Metric
- removed R77: 100, Resistor_SMD:R_0805_2012Metric
- removed U17: NCA9555, Package_SO:TSSOP-24_4.4x7.8mm_P0.65mm
- added C43: 0.1u, Capacitor_SMD:C_0805_2012Metric, F.Cu at (111.5, 88.0)
- added C44: 0.1u, Capacitor_SMD:C_0805_2012Metric, F.Cu at (189.5, 12.2)
- added C45: 0.1u, Capacitor_SMD:C_0805_2012Metric, F.Cu at (189.5, 2.00)
- added C46: 1u, Capacitor_SMD:C_0805_2012Metric, F.Cu at (104.8, 67.5)
- added C47: 0.1u, Capacitor_SMD:C_0805_2012Metric, F.Cu at (200.1, 27.8)
- added J31: CAN, Connector_JST:JST_PH_B4B-PH-K_1x04_P2.00mm_Vertical, B.Cu at (102.5, 48.0)
- added J37: SKP OUT, Connector_JST:JST_PH_B2B-PH-K_1x02_P2.00mm_Vertical, B.Cu at (102.5, 59.2)
- added J40: Door Closed, Connector_JST:JST_PH_B2B-PH-K_1x02_P2.00mm_Vertical, B.Cu at (102.5, 66.5)
- added J46: Conn_01x16_Pin, Connector_PinHeader_2.54mm:PinHeader_1x16_P2.54mm_Vertical, F.Cu at (102.0, 73.0)
- added R61: 0, Resistor_SMD:R_0805_2012Metric, B.Cu at (58.5, 106.4)
- added R62: 10k, Resistor_SMD:R_0805_2012Metric, F.Cu at (109.8, 67.5)
- added R63: 10k, Resistor_SMD:R_0805_2012Metric, F.Cu at (198.7, 17.2)
- added R64: 100, Resistor_SMD:R_0805_2012Metric, F.Cu at (107.2, 67.5)
- added R65: 0, Resistor_SMD:R_0805_2012Metric, B.Cu at (65.2, 83.8)
- added U13: NCA9555, Package_SO:TSSOP-24_4.4x7.8mm_P0.65mm, F.Cu at (109.0, 82.8)
- C40: value 4.7n -> 0.1u
- C42: value 0.1u -> 4.7n
- J43: value Door Closed -> Servo A; footprint Connector_JST:JST_PH_B2B-PH-K_1x02_P2.00mm_Vertical -> Connector_JST:JST_PH_B3B-PH-K_1x03_P2.00mm_Vertical
- J44: value CAN -> Servo B; footprint Connector_JST:JST_PH_B4B-PH-K_1x04_P2.00mm_Vertical -> Connector_JST:JST_PH_B3B-PH-K_1x03_P2.00mm_Vertical
- R35, R39, R60: moved to B.Cu
- U14: value NCA9555 -> SN74HC14DR; footprint Package_SO:TSSOP-24_4.4x7.8mm_P0.65mm -> Package_SO:SOIC-14_3.9x8.7mm_P1.27mm
- U16: value SN74HC14DR -> NCA9555; footprint Package_SO:SOIC-14_3.9x8.7mm_P1.27mm -> Package_SO:TSSOP-24_4.4x7.8mm_P0.65mm
- moved C33 443.1 mm to (74.7, 141.7)
- moved C34 443.1 mm to (72.2, 148.0)
- moved D15 443.1 mm to (71.9, 132.2)
- moved R53 443.1 mm to (71.9, 136.7)
- moved SW3 443.1 mm to (65.2, 136.5)
- moved TP22 443.1 mm to (75.7, 129.0)
- moved TP23 443.1 mm to (69.2, 129.0)
- moved U10 443.1 mm to (70.7, 143.0)
- moved C20 332.4 mm to (195.7, 140.5)
- moved C21 332.4 mm to (195.7, 143.5)
- moved U14 301.6 mm to (195.5, 13.8), turned to 90 degrees
- moved C29 147.0 mm to (114.5, 134.5)
- moved C28 140.5 mm to (108.2, 129.8), turned to 180 degrees
- moved C42 126.4 mm to (117.2, 65.8), turned to -90 degrees
- moved U16 123.8 mm to (211.2, 11.0), turned to 90 degrees
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Connections:
- C40 pad 1: Net-(C40-Pad1) -> GND
- C40 pad 2: GND -> Net-(U12-IN-)
- C42 pad 1: /Display/DISP_3V3 -> Net-(C42-Pad1)
- F1 pad 2: /R3V3 -> /SYS5V0
- J43 pad 1: GND -> /Servos/SRV_5V0
- J43 pad 2: Net-(J43-Pin_2) -> GND
- J44 pad 1: /CAN/CAN- -> (no net)
- J44 pad 2: /CAN/CAN+ -> (no net)
- J44 pad 3: GND -> (no net)
- J45 pad 1: /R3V3 -> /SYS5V0
- J47 pad 1: /Display/IO0 -> /Buttons/IN0
- J47 pad 10: /Display/IO9 -> /Encoder/IN9
- J47 pad 11: /Display/IO10 -> /Encoder/IN10
- J47 pad 12: /Display/IO11 -> unconnected-(J47-Pin_12-Pad12)
- J47 pad 13: /Display/IO12 -> unconnected-(J47-Pin_13-Pad13)
- J47 pad 14: /Display/IO13 -> unconnected-(J47-Pin_14-Pad14)
- J47 pad 15: /Display/IO14 -> unconnected-(J47-Pin_15-Pad15)
- J47 pad 16: /Display/IO15 -> unconnected-(J47-Pin_16-Pad16)
- J47 pad 2: /Display/IO1 -> /Buttons/IN1
- J47 pad 3: /Display/IO2 -> /Buttons/IN2
- J47 pad 4: /Display/IO3 -> /Buttons/IN3
- J47 pad 5: /Display/IO4 -> /Buttons/IN4
- J47 pad 6: /Display/IO5 -> /Buttons/IN5
- J47 pad 7: /Display/IO6 -> /Buttons/IN6
- J47 pad 8: /Display/IO7 -> /Buttons/IN7
- J47 pad 9: /Display/IO8 -> /Encoder/IN8
- R35 pad 2: /R3V3 -> /SYS5V0
- R46 pad 2: /R3V3 -> /SYS5V0
- R56 pad 2: /R3V3 -> /SYS5V0
- R57 pad 2: Net-(C40-Pad1) -> Net-(C41-Pad1)
- R58 pad 1: Net-(C40-Pad1) -> Net-(C41-Pad1)
- R58 pad 2: Net-(C41-Pad1) -> Net-(C42-Pad1)
- R6 pad 2: /R3V3 -> /SYS5V0
- R66 pad 1: /Buttons/BTN_3V3 -> /Servos/SRV_5V0
- R66 pad 2: /R3V3 -> /SYS5V0
- R7 pad 2: /R3V3 -> /SYS5V0
- RV1 pad 1: Net-(C41-Pad1) -> Net-(C42-Pad1)
- TP2 pad 1: /R3V3 -> /SYS5V0
- U14 pad 1: unconnected-(U14-~{INT}-Pad1) -> /Buttons/IN0
- U14 pad 10: /Display/IO6 -> /Buttons/BTN4
- U14 pad 11: /Display/IO7 -> /Buttons/IN4
- U14 pad 12: GND -> /Buttons/BTN5
- U14 pad 13: /Display/IO8 -> /Buttons/IN5
- U14 pad 14: /Display/IO9 -> /Buttons/BTN_3V3
- U14 pad 2: GND -> /Buttons/BTN0
- U14 pad 3: GND -> /Buttons/IN1
- U14 pad 4: /Display/IO0 -> /Buttons/BTN1
- U14 pad 5: /Display/IO1 -> /Buttons/IN2
- U14 pad 6: /Display/IO2 -> /Buttons/BTN2
- U14 pad 7: /Display/IO3 -> GND
- U14 pad 8: /Display/IO4 -> /Buttons/BTN3
- U14 pad 9: /Display/IO5 -> /Buttons/IN3
- U15 pad 1: /Buttons/IN0 -> /Buttons/IN6
- U15 pad 10: /Buttons/BTN4 -> /Encoder/ENC.B
- U15 pad 11: /Buttons/IN4 -> /Encoder/IN10
- U15 pad 12: /Buttons/BTN5 -> /Buttons/DoorLS
- U15 pad 13: /Buttons/IN5 -> Net-(C46-Pad1)
- U15 pad 2: /Buttons/BTN0 -> /Buttons/BTN6
- U15 pad 3: /Buttons/IN1 -> /Buttons/IN7
- U15 pad 4: /Buttons/BTN1 -> /Buttons/BTN7
- U15 pad 5: /Buttons/IN2 -> /Encoder/IN8
- U15 pad 6: /Buttons/BTN2 -> /Encoder/ENC.SW
- U15 pad 8: /Buttons/BTN3 -> /Encoder/ENC.A
- U15 pad 9: /Buttons/IN3 -> /Encoder/IN9
- U16 pad 1: /Buttons/IN6 -> /Buttons/~{BTN_IRQ}
- U16 pad 10: /Encoder/ENC.B -> /Buttons/BTN6
- U16 pad 11: /Encoder/IN10 -> /Buttons/BTN7
- U16 pad 12: /Buttons/DoorLS -> GND
- U16 pad 13: Net-(C57-Pad1) -> /Buttons/LED0
- U16 pad 14: /Buttons/BTN_3V3 -> /Buttons/LED1
- U16 pad 2: /Buttons/BTN6 -> GND
- U16 pad 3: /Buttons/IN7 -> GND
- U16 pad 4: /Buttons/BTN7 -> /Buttons/BTN0
- U16 pad 5: /Encoder/IN8 -> /Buttons/BTN1
- U16 pad 6: /Encoder/ENC.SW -> /Buttons/BTN2
- U16 pad 7: GND -> /Buttons/BTN3
- U16 pad 8: /Encoder/ENC.A -> /Buttons/BTN4
- U16 pad 9: /Encoder/IN9 -> /Buttons/BTN5
Routing:
- net /Display/IO0: track 21.9 -> 0.00 mm
- net /Display/IO1: track 19.3 -> 0.00 mm
- net /Display/IO2: track 16.5 -> 0.00 mm
- net /Display/IO3: track 14.3 -> 0.00 mm
- net /Display/IO4: track 10.7 -> 0.00 mm
- net /Display/IO5: track 8.02 -> 0.00 mm
- net /Display/IO6: track 5.15 -> 0.00 mm

Commit message: progress save for the night. landmarking of service PCB is almost done. redid the analog section layout to make it more assembleable and better utilze the space. Still need to do ACC, R3V3, IO, test points, and jumpers
Parts:
- removed R65: 0, Resistor_SMD:R_0805_2012Metric
- D13, D14, D3, D4, D5, D6, D7, D8, R1, R12, R13, R14, R17, R18, R19, R25, R30, R31, R46, R48, R5, R54, R55, R56, R6, R66, R7, R8, R9: moved to B.Cu
- J47: footprint Connector_PinHeader_2.54mm:PinHeader_1x16_P2.54mm_Vertical -> Connector_PinHeader_2.54mm:PinHeader_1x19_P2.54mm_Vertical
- R37: value 10k -> 20k
- moved R23 203.1 mm to (67.0, 130.2)
- moved R24 203.1 mm to (67.0, 133.3)
- moved TP25 202.8 mm to (58.5, 28.2)
- moved TP26 202.8 mm to (58.5, 32.3)
- moved F1 194.0 mm to (149.8, 61.0), turned to 90 degrees
- moved R9 172.2 mm to (120.2, 104.5)
- moved TP24 169.2 mm to (68.0, 75.2)
- moved R56 161.1 mm to (39.4, 76.5)
- moved R48 160.2 mm to (33.1, 75.5)
- moved R46 159.7 mm to (33.1, 81.4)
- moved R55 159.6 mm to (39.4, 79.5)
- moved TP12 155.8 mm to (60.0, 48.5)
- moved TP13 155.8 mm to (60.0, 53.1)
- moved TP14 155.8 mm to (60.0, 57.8)
- moved R25 136.3 mm to (45.1, 72.8)
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Connections:
- net /Buttons/LED0 renamed /Buttons/IO16
- net /Buttons/LED1 renamed /Buttons/IO17
- net /Buttons/LED2 renamed /Buttons/IO18
- net /Buttons/LED3 renamed /Buttons/IO19
- net /Buttons/LED4 renamed /Buttons/IO20
- net /Buttons/LED5 renamed /Buttons/IO21
- net /Buttons/LED6 renamed /Buttons/IO22
- net /Buttons/LED7 renamed /Buttons/IO23
- J15 pad 10: /MCU/DoorLS -> /Buttons/DoorLS
- J19 pad 1: /Load Cell/E+ -> /Load Cell/A-
- J19 pad 2: /Load Cell/E- -> /Load Cell/A+
- J19 pad 3: /Load Cell/A+ -> /Load Cell/E-
- J19 pad 4: /Load Cell/A- -> /Load Cell/E+
- J44 pad 1: (no net) -> /Servos/SRV_5V0
- J44 pad 2: (no net) -> GND
- J44 pad 3: (no net) -> /MCU/SRV.B
- J47 pad 12: unconnected-(J47-Pin_12-Pad12) -> /Stackup Header/IO16
- J47 pad 13: unconnected-(J47-Pin_13-Pad13) -> /Stackup Header/IO17
- J47 pad 14: unconnected-(J47-Pin_14-Pad14) -> /Stackup Header/IO18
- J47 pad 15: unconnected-(J47-Pin_15-Pad15) -> /Stackup Header/IO19
- J47 pad 16: unconnected-(J47-Pin_16-Pad16) -> /Stackup Header/IO20
- U6 pad 24: /MCU/DoorLS -> /Buttons/DoorLS
- U8 pad 8: unconnected-(U8-EN/~{CAL}-Pad8) -> /MCU/ESP32_25
Routing:
- net /CAN/CAN-: track 66.3 -> 50.3 mm
- net /Display/IO7: track 0.00 -> 15.2 mm
- net /Display/IO6: track 0.00 -> 13.9 mm
- net /Display/IO5: track 0.00 -> 12.5 mm
- net /Display/IO0: track 0.00 -> 11.9 mm
- net /Display/IO4: track 0.00 -> 11.4 mm
- net /Display/IO3: track 0.00 -> 10.2 mm
- net /Display/IO1: track 0.00 -> 10.2 mm
- net /CAN/CAN+: track 63.3 -> 54.0 mm
- net /Display/IO2: track 0.00 -> 9.35 mm
- added copper zone on In1.Cu, net GNDA
Other:
- board size 205 x 104.8 mm -> 70 x 90 mm
