File: KiCAD/LiF_FC-PCB_rev1/LiF_MCU.kicad_sch (KiCad schematic)
At the start: 38 parts, among them J12 ESP 3V3_{EN}, J13 ESP_DGB_CONN, J14 CAN Upstream, J15 ESP_DGB_CONN, J16 ESP_DGB_CONN, Q1 MMBT4401, Q2 MMBT4401, SW1 Flash, SW2 Reset, U6 ESP32-S3-WROOM-1, U7 CY7C65213-28PVXI

Commit message: backup before leaving school
Parts:
- J12: footprint Connector_PinHeader_2.54mm:PinHeader_1x02_P2.54mm_Vertical -> Connector_PinHeader_2.54mm:PinHeader_1x02_P2.54mm_Vertical_SMD_Pin1Left
Changed lines of the file:
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@@
 			)
 		)
-		(property "Footprint" "Connector_PinHeader_2.54mm:PinHeader_1x02_P2.54mm_Vertical"
+		(property "Footprint" "Connector_PinHeader_2.54mm:PinHeader_1x02_P2.54mm_Vertical_SMD_Pin1Left"
 			(at 44.45 40.64 0)
 			(effects

Commit message: progress backup before increasing the size of the PCB again
Connections:
- net ESP32_36: now also U6.36 (RXD0), U7.1 (TXD); no longer U6.37 (TXD0), U7.5 (RXD)
- net ESP32_37: now also U6.37 (TXD0), U7.5 (RXD); no longer U6.36 (RXD0), U7.1 (TXD)
- net D+ renamed USB.D+
- net D- renamed USB.D-
Changed lines of the file:
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@@
-		)
-	)
-	(label "ESP32_37"
-		(at 231.14 69.85 180)
-		(effects
-			(font
-				(size 1.27 1.27)
-			)
-			(justify right bottom)
 		)
 	)
@@
 		)
 	)
-	(label "D-"
+	(label "USB.D-"
 		(at 74.93 101.6 0)
 		(effects
@@
 			)
 			(justify left bottom)
-		)
-	)
-	(label "ESP32_36"
-		(at 231.14 67.31 180)
-		(effects
-			(font
-				(size 1.27 1.27)
-			)
-			(justify right bottom)
 		)
 	)
@@
 		)
 	)
+	(label "ESP32_37"
+		(at 231.14 67.31 180)
+		(effects
+			(font
+				(size 1.27 1.27)
+			)
+			(justify right bottom)
+		)
+	)
 	(label "ESP32_39"
 		(at 137.16 74.93 0)
@@
 		)
 	)
-	(label "D+"
+	(label "USB.D+"
 		(at 49.53 149.86 0)
 		(effects
@@
 		)
 	)
+	(label "ESP32_36"
+		(at 231.14 69.85 180)
+		(effects
+			(font
+				(size 1.27 1.27)
+			)
+			(justify right bottom)
+		)
+	)
 	(label "ESP32_5"
 		(at 262.89 50.8 0)
@@
 		)
 	)
-	(label "D-"
+	(label "USB.D-"
 		(at 49.53 152.4 0)
 		(effects
@@
 		)
 	)
-	(label "D+"
+	(label "USB.D+"
 		(at 74.93 95.25 0)
 		(effects

Commit message: Created new KiCAD project for IO PCB, moved relevant components there, saving backup before reannotating the Service PCB schematics
Parts:
- J12: now not fitted; now left out of the parts list

Commit message: progress save for the night. landmarking of service PCB is almost done. redid the analog section layout to make it more assembleable and better utilze the space. Still need to do ACC, R3V3, IO, test points, and jumpers
Connections:
- net ESP32_25 renamed IA_EN
Other:
- note removed: "free to use"
Changed lines of the file:
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@@
 		)
 	)
-	(text "free to use"
-		(exclude_from_sim no)
-		(at 237.744 112.268 0)
-		(effects
-			(font
-				(size 1.27 1.27)
-			)
-		)
-	)
 	(text "PSRAM"
 		(exclude_from_sim no)
@@
 	(wire
 		(pts
-			(xy 201.93 113.03) (xy 231.14 113.03)
+			(xy 201.93 113.03) (xy 242.57 113.03)
 		)
 		(stroke
@@
 	(wire
 		(pts
+			(xy 243.84 26.67) (xy 254 26.67)
+		)
+		(stroke
+			(width 0)
+			(type default)
+		)
+	)
+	(wire
+		(pts
 			(xy 83.82 106.68) (xy 83.82 95.25)
 		)
@@
 		)
 	)
+	(label "IA_{EN}"
+		(at 254 26.67 180)
+		(effects
+			(font
+				(size 1.27 1.27)
+			)
+			(justify right bottom)
+		)
+	)
 	(label "ESP32_28"
 		(at 231.14 85.09 180)
@@
 		)
 	)
+	(label "IA_{EN}"
+		(at 242.57 113.03 180)
+		(effects
+			(font
+				(size 1.27 1.27)
+			)
+			(justify right bottom)
+		)
+	)
 	(label "DTR"
 		(at 95.25 165.1 180)
@@
 		(effects
 			(font
+				(size 1.27 1.27)
+			)
+			(justify right)
+		)
+	)
+	(hierarchical_label "IA_EN"
+		(shape output)
+		(at 243.84 26.67 180)
+		(effects
+			(font

Commit message: finished service PCB routing and silkscreen, finished IO PCB layout, routing, and silkscreen. Exported production files, submitted PCB for manufacturing by JLCPCB
Parts:
- R23, R24, R26, R27, R28, R29, R30, R31, R32, R33: footprint Capacitor_SMD:C_0805_2012Metric -> Resistor_SMD:R_0805_2012Metric
Changed lines of the file:
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@@
 		)
 	)
+	(label "V_{ST}.SYS"
+		(at 243.84 74.93 180)
+		(effects
+			(font
+				(size 1.27 1.27)
+			)
+			(justify right bottom)
+		)
+	)
 	(label "ESP_3V3"
 		(at 24.13 143.51 180)
@@
 		)
 	)
-	(label "V_{ST}.SYS"
-		(at 243.84 72.39 180)
-		(effects
-			(font
-				(size 1.27 1.27)
-			)
-			(justify right bottom)
-		)
-	)
 	(label "ESP32_18"
 		(at 137.16 97.79 0)
@@
 		)
 	)
+	(label "V_{ST}.AUX"
+		(at 243.84 72.39 180)
+		(effects
+			(font
+				(size 1.27 1.27)
+			)
+			(justify right bottom)
+		)
+	)
 	(label "ESP32_33"
 		(at 231.14 97.79 180)
@@
 		)
 	)
-	(label "V_{ST}.AUX"
-		(at 243.84 74.93 180)
-		(effects
-			(font
-				(size 1.27 1.27)
-			)
-			(justify right bottom)
-		)
-	)
 	(label "ESP32_31"
 		(at 262.89 129.54 0)
@@
 			)
 		)
-		(property "Footprint" "Capacitor_SMD:C_0805_2012Metric"
+		(property "Footprint" "Resistor_SMD:R_0805_2012Metric"
 			(at 21.082 110.49 90)
 			(effects
@@
 			)
 		)
-		(property "Footprint" "Capacitor_SMD:C_0805_2012Metric"
+		(property "Footprint" "Resistor_SMD:R_0805_2012Metric"
 			(at 93.218 144.78 90)
 			(effects
@@
 			)
 		)
-		(property "Footprint" "Capacitor_SMD:C_0805_2012Metric"
+		(property "Footprint" "Resistor_SMD:R_0805_2012Metric"
 			(at 29.718 110.49 90)
 			(effects
@@
 			)
 		)
-		(property "Footprint" "Capacitor_SMD:C_0805_2012Metric"
+		(property "Footprint" "Resistor_SMD:R_0805_2012Metric"
 			(at 43.688 157.48 90)
 			(effects
@@
 			)
 		)
-		(property "Footprint" "Capacitor_SMD:C_0805_2012Metric"
+		(property "Footprint" "Resistor_SMD:R_0805_2012Metric"
 			(at 125.73 179.578 90)
 			(effects
@@
 			)
 		)
-		(property "Footprint" "Capacitor_SMD:C_0805_2012Metric"
+		(property "Footprint" "Resistor_SMD:R_0805_2012Metric"
 			(at 130.302 34.29 90)
 			(effects
@@
 			)
 		)
-		(property "Footprint" "Capacitor_SMD:C_0805_2012Metric"
+		(property "Footprint" "Resistor_SMD:R_0805_2012Metric"
 			(at 137.668 34.29 90)
 			(effects
@@
 			)
 		)
-		(property "Footprint" "Capacitor_SMD:C_0805_2012Metric"
+		(property "Footprint" "Resistor_SMD:R_0805_2012Metric"
 			(at 164.338 146.05 90)
 			(effects
@@
 			)
 		)
-		(property "Footprint" "Capacitor_SMD:C_0805_2012Metric"
+		(property "Footprint" "Resistor_SMD:R_0805_2012Metric"
 			(at 125.73 160.528 90)
 			(effects
@@
 			)
 		)
-		(property "Footprint" "Capacitor_SMD:C_0805_2012Metric"
+		(property "Footprint" "Resistor_SMD:R_0805_2012Metric"
 			(at 33.528 157.48 90)
 			(effects
