File: KiCAD/LiF_FC-PCB_rev1/LiF_Servos.kicad_sch (KiCad schematic)
At the start: 6 parts, among them J42 SRV 3V3_{EN}, J43 Servo A, J44 Servo B

Commit message: finished service PCB routing and silkscreen, finished IO PCB layout, routing, and silkscreen. Exported production files, submitted PCB for manufacturing by JLCPCB
Parts:
- removed TP30: SRV_{A}, TestPoint:TestPoint_Loop_D1.80mm_Drill1.0mm_Beaded, symbol Connector:TestPoint
- removed TP31: SRV_{B}, TestPoint:TestPoint_Loop_D1.80mm_Drill1.0mm_Beaded, symbol Connector:TestPoint
Connections:
- net SRV.A: now also J43.1 (Pin_1); no longer J43.3 (Pin_3)
- net SRV.B: now also J44.1 (Pin_1); no longer J44.3 (Pin_3)
- net SRV_5V0: now also J43.3 (Pin_3), J44.3 (Pin_3); no longer J43.1 (Pin_1), J44.1 (Pin_1)
